File: beacon1.brd (EAGLE design)
At the start: 111.7 x 103.8 mm, 108 parts, among them IC1 NCP1117ST50T3G, IC6 LP2985-33DBVR, IC7 LMV358IDGKR, SW1 EG1319, T1 FDN340P, U1 FGPMMOPA6H, U2 MIC5225-3.3, U4 MIC5225-3.3, U5 MB85RC256VPF-G-JNERE2, X1 JST 2PH, Y1 CSTCE16M0V53-R0 16MHZ, Y2 32.768kHz (535-9166-2-ND)

Commit message: redid layout, might be better for routing?
Parts:
- moved R41 105.2 mm to (106.7, 14.0), turned to 270 degrees
- moved R36 104.3 mm to (8.89, -1.27)
- moved Y1 101.3 mm to (106.7, 21.6)
- moved IC6 96.1 mm to (16.5, -1.27)
- moved R3 94.6 mm to (27.9, 2.54), turned to 180 degrees
- moved R4 93.7 mm to (66.0, 2.54), turned to 90 degrees
- moved USB_1 93.2 mm to (55.9, 1.27)
- moved C1 92.2 mm to (38.1, 14.0), turned to 90 degrees
- moved C2 92.0 mm to (34.3, 12.7), turned to 90 degrees
- moved C16 90.9 mm to (25.4, -1.27)
- moved 3V3_ON_LED 89.7 mm to (2.54, -1.27)
- moved 5V_ON_LED 88.9 mm to (26.7, 48.3)
- moved L1 85.2 mm to (44.5, -1.27)
- moved C15 82.5 mm to (78.7, 22.9)
- moved PC2 79.8 mm to (33.0, 24.1), turned to 180 degrees
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Other:
- board size 111.7 x 103.8 mm -> 111.7 x 105.1 mm

Commit message: almost 100% routed, but with a lot of gross vias
Routing:
- net 90348: track 0.00 -> 614.1 mm, vias 0 -> 4
- net GND: track 0.00 -> 504.1 mm, vias 0 -> 4
- net 5V: track 0.00 -> 409.6 mm, vias 0 -> 12
- net VIN: track 0.00 -> 257.2 mm, vias 0 -> 4
- net 3.3V: track 0.00 -> 181.2 mm, vias 0 -> 4
- net 3V3: track 0.00 -> 153.2 mm, vias 0 -> 1
- net RESET: track 0.00 -> 140.7 mm, vias 0 -> 1
- net N$120: track 0.00 -> 132.0 mm, vias 0 -> 2
- net CTS_3V: track 0.00 -> 128.5 mm, vias 0 -> 3
- net N$21: track 0.00 -> 111.8 mm, vias 0 -> 5
- net SDA: track 0.00 -> 103.1 mm, vias 0 -> 2
- net RXD_3V: track 0.00 -> 98.7 mm, vias 0 -> 2
- net XTAL2: track 0.00 -> 96.9 mm
- net SCL: track 0.00 -> 94.3 mm, vias 0 -> 3
- net CMP: track 0.00 -> 87.1 mm
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Other:
- board size 111.7 x 105.1 mm -> 113 x 112.7 mm

Commit message: save before leaving for meeting
Parts:
- moved D11 13.0 mm to (30.5, 74.9)
- moved 3V3_REV_LED 13.0 mm to (21.6, 58.4)
- moved 5V_ON_LED 13.0 mm to (29.2, 61.0)
- moved 5V_REV_LED 13.0 mm to (99.1, 108.0)
- moved ATMEGA2560 13.0 mm to (58.4, 58.4)
- moved B1 13.0 mm to (35.6, 49.5)
- moved C10 13.0 mm to (47.0, 99.1)
- moved C11 13.0 mm to (44.5, 67.3)
- moved C13 13.0 mm to (88.9, 38.1)
- moved C15 13.0 mm to (81.3, 35.6)
- moved C6 13.0 mm to (53.3, 72.4)
- moved C8 13.0 mm to (47.0, 88.9)
- moved C9 13.0 mm to (47.0, 94.0)
- moved D10 13.0 mm to (39.4, 104.1)
- moved D12 13.0 mm to (22.9, 105.4)
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