File: beacon1.sch (EAGLE design)
At the start: 15 parts, among them U1 FGPMMOPA6H, U2 MIC5225-3.3

Commit message: added atmega 2560 to schematic
Parts:
- added 3V3_ON_LED, 5V_ON_LED, PWRIN_ON_LED, USB_POWER_ON_LED: GREEN, SparkFun-LED:LED-GREENLILYPAD
- added 3V3_REV_LED, 5V_REV_LED, PWRIN_REV_LED: RED, SparkFun-LED:LED-RED1206
- added ATMEGA2560: ATMEGA2560-16AU, SparkFun-DigitalIC:ATMEGA2560AU
- added C10, C12, C14, C15, C16, C6, C7, C8, C9: 100n, SmartPrj:C-EUC1206K
- added C11: 22p, SmartPrj:C-EUC1206K
- added C13: 1u, SmartPrj:C-EUC1206K
- added C4, C5: (no value), eagle-ltspice:CC1206
- added D3: M7, diode:DIODE-SMB
- added D4: CD1206-S01575, diode:DIODE-MINIMELF
- added F1: MF-MSMF050-2 500mA, rcl:L-EUL1812
- added FTDI: FT232RL, ftdichip:FT232RL
- added FTDI_RESET: TEST-POINT2, SparkFun-Connectors:TEST-POINT2
- added IC1: NCP1117ST50T3G, linear:MC33269ST-3.3T3
- added IC6: LP2985-33DBVR, SmartPrj:LP2985-XXDBVR33
- added IC7: LMV358IDGKR, linear:LMV358MMX
- added ICSP: 3x2M, SmartPrj:PINHD-2X3
- added L: YELLOW, SparkFun-LED:LED1206
- added L1: BLM21, wuerth-elektronik:WE-CBF_0805
- added LED2: (no value), microbuilder:LED1206
- added MICRO_SD_1: MICRO-SD_CARD_SOCKET, SparkFun-Connectors:MICRO-SD_CARD_SOCKET
- added PC1, PC2: 47u, rcl:CPOL-EUD
- added Q4, Q5, Q6, Q7: 220mA/50V/3.5Ω, SparkFun-DiscreteSemi:MOSFET-NCH-BSS138
- added R10, R8, R9: 1k, adafruit:R-US_M1206
- added R11, R12, R13, R6, R7: 10k, adafruit:R-US_M1206
- added R36, R37, R38, R39, R40, R41, R54: (no value), resistor:R-US_M1206
- added R4: 1K, microbuilder:RESISTOR0805_NOOUTLINE
- added R42, R43, R44, R45, R46, R47, R48, R49: (no value), rcl:R-US_M1206
- added R5: 1M, SmartPrj:R-EU_R1206
- added RESET: TS42031-160R-TR-7260, SmartPrj:TS42
- added RX, TX: YELLOW, led:LEDSMT1206
- added T1: FDN340P, zetex:PMOSSOT23
- added U$1: XBEE, adafruit:XBEE
- added USB_1: USB-B_TH, SmartPrj:PN61729
- added Y1: CSTCE16M0V53-R0 16MHZ, SmartPrj:RESONATORMU
- added Z1, Z2: CG0603MLC-05E, varistor:VARISTORCN0603
Connections:
- new net 3V3: 3V3_ON_LED.A, C13.2, C4.1, C5.1, IC6.OUT, IC7B.-IN, MICRO_SD_1.VCC, Q4.G, Q5.G, Q6.G, Q7.G, R36.1, R42.2, R44.2, R46.2, R48.2, U$1.VCC
- new net 5V: 5V_ON_LED.A, ATMEGA2560.AVCC, ATMEGA2560.VCC, ATMEGA2560.VCC1, ATMEGA2560.VCC2, ATMEGA2560.VCC3, C10.1, C14.1, C16.2, C7.1, C9.1, D4.C, FTDI.VCC, FTDI.VCCIO, IC1.OUT, IC1.OUT@1, IC6.IN, IC6.ON/!OFF, IC7P.V+, ICSP.2, PC2.+, R11.1, R12.1, R13.1, R37.1, R43.2, R45.2, R47.2, R49.2, R8.2, R9.2, T1.S
- new net 90348: 3V3_REV_LED.A, 5V_REV_LED.A, ATMEGA2560.AGND, ATMEGA2560.GND, ATMEGA2560.GND1, ATMEGA2560.GND2, ATMEGA2560.GND3, C10.2, C11.2, C12.2, C13.1, C14.2, C15.1, C16.1, C6.2, C7.2, C8.2, C9.2, FTDI.GND@1, FTDI.GND@A, IC1.GND/ADJ, IC6.GND, IC7P.V-, ICSP.6, L.C, L1.1, MICRO_SD_1.CD2, MICRO_SD_1.GND, MICRO_SD_1.SHIELD@1, MICRO_SD_1.SHIELD@3, PC1.-, PC2.-, PWRIN_REV_LED.A, R38.1, R39.1, R40.1, R41.1, R7.1, RESET.1, RESET.2, USB_1.4, Y1.2
- new net ADC0: ATMEGA2560.(ADC0)PF0
- new net ADC1: ATMEGA2560.(ADC1)PF1
- new net ADC10: ATMEGA2560.PK2(ADC10/PCINT18)
- new net ADC11: ATMEGA2560.PK3(ADC11/PCINT19)
- new net ADC12: ATMEGA2560.PK4(ADC12/PCINT20)
- new net ADC13: ATMEGA2560.PK5(ADC13/PCINT21)
- new net ADC14: ATMEGA2560.PK6(ADC14/PCINT22)
- new net ADC15: ATMEGA2560.PK7(ADC15/PCINT23)
- new net ADC2: ATMEGA2560.(ADC2)PF2
- new net ADC3: ATMEGA2560.(ADC3)PF3
- new net ADC4: ATMEGA2560.(ADC4/TCK)PF4
- new net ADC5: ATMEGA2560.(ADC5/TMS)PF5
- new net ADC6: ATMEGA2560.(ADC6/TDO)PF6
- new net ADC7: ATMEGA2560.(ADC7/TDI)PF7
- new net ADC8: ATMEGA2560.PK0(ADC8/PCINT16)
- new net ADC9: ATMEGA2560.PK1(ADC9/PCINT17)
- new net ADO: ATMEGA2560.PJ7
- new net AREF: ATMEGA2560.AREF, C6.1
- new net CAN_CS: ATMEGA2560.PL2(T5)
- new net CAN_INT: ATMEGA2560.PJ4(PCINT13)
- new net CAN_RESET: ATMEGA2560.PH3(OC4A)
- new net CAN_RX0BF: ATMEGA2560.PL6
- new net CAN_RX1BF: ATMEGA2560.PL7
- new net CAN_TX0RTS: ATMEGA2560.PL3(OC5A)
- new net CAN_TX1RTS: ATMEGA2560.PL4(OC5B)
- new net CAN_TX2RTS: ATMEGA2560.PL5(OC5C)
- new net CMP: C15.2, IC7B.+IN, R6.1, R7.2
- new net D+: FTDI.USBDP, USB_1.3, Z2.2
- new net D-: FTDI.USBDM, USB_1.2, Z1.2
- new net GATE_CMD: IC7B.OUT, T1.G
- new net IMU_CS_HI: ATMEGA2560.PL0(ICP4)
- new net IMU_INT_HI: ATMEGA2560.PJ5(PCINT14)
- new net L13: IC7A.-IN, IC7A.OUT, R10.2
- new net LED0: ATMEGA2560.(A8)PC0
- new net LED1: ATMEGA2560.(A9)PC1
- new net LED10: ATMEGA2560.(AD2)PA2
- new net LED11: ATMEGA2560.(AD3)PA3
- new net LED12: ATMEGA2560.(AD4)PA4
- new net LED13: ATMEGA2560.(AD5)PA5
- new net LED14: ATMEGA2560.(AD6)PA6
- new net LED15: ATMEGA2560.(AD7)PA7
- new net LED2: ATMEGA2560.(A10)PC2
- new net LED3: ATMEGA2560.(A11)PC3
- new net LED4: ATMEGA2560.(A12)PC4
- new net LED5: ATMEGA2560.(A13)PC5
- new net LED6: ATMEGA2560.(A14)PC6
- new net LED7: ATMEGA2560.(A15)PC7
- new net LED8: ATMEGA2560.(AD0)PA0
- new net LED9: ATMEGA2560.(AD1)PA1
- new net MISO: ATMEGA2560.(MISO/PCINT3)PB3, ICSP.1, Q5.D, R45.1
- new net MOSI: ATMEGA2560.(MOSI/PCINT2)PB2, ICSP.4, Q4.D, R43.1
- new net N$11: 5V_REV_LED.C, FTDI.CBUS2, R37.2
- new net N$12: 3V3_ON_LED.C, FTDI.CBUS3, R39.2
- new net N$13: PWRIN_ON_LED.C, R40.2
- new net N$14: R41.2, USB_POWER_ON_LED.C
- new net N$20: PWRIN_REV_LED.C, R54.2
- new net N$37: 3V3_REV_LED.C, R36.2
- new net N$48: 5V_ON_LED.C, R38.2
- new net N$54: R9.1, RX.A
- new net N$55: R8.1, TX.A
- new net N$6: LED2.A, R4.2
- new net N$60: U$1.DO8
- new net N$61: U$1.RESET
- new net N$63: U$1.PWM1
- new net N$64: U$1.RESERVED
- new net N$65: U$1.DTR/DI8
- new net N$66: U$1.AD0/DIO0
- new net N$67: U$1.AD1/DIO1
- new net N$68: U$1.AD2/DIO2
- new net N$69: U$1.AD3/DIO3
- new net N$7: L.A, R10.1
- new net N$70: U$1.RTS/AD6/DIO6
- new net N$71: R4.1, U$1.ASC/AD5/DIO5
- new net N$72: U$1.VREF
- new net N$73: U$1.ON/SLEEP
- new net N$74: U$1.CTS/DIO7
- new net N$75: U$1.AD4/DIO4
- new net N$8: FTDI.GND, FTDI.GND@2, FTDI.TEST
- new net N$9: FTDI.!RESET, FTDI_RESET.1
- new net PB0: ATMEGA2560.(SS/PCINT0)PB0
- new net PB4: ATMEGA2560.(OC2A/PCINT4)PB4
- new net PB5: ATMEGA2560.(OC1A/PCINT5)PB5
- new net PB6: ATMEGA2560.(OC1B/PCINT6)PB6
- new net PB7: ATMEGA2560.(OC0A/OC1C/PCINT7)PB7, IC7A.+IN
- new net PD7: ATMEGA2560.(T0)PD7
- new net PE3: ATMEGA2560.(OC3A/AIN1)PE3
- new net PE4: ATMEGA2560.(OC3B/INT4)PE4
- new net PE5: ATMEGA2560.(OC3C/INT5)PE5
- new net PE6: ATMEGA2560.(T3/INT6)PE6
- new net PE7: ATMEGA2560.(CLKO/ICP3/INT7)PE7
- new net PG0: ATMEGA2560.(WR)PG0
- new net PG1: ATMEGA2560.(RD)PG1
- new net PG2: ATMEGA2560.(ALE)PG2
- new net PG5: ATMEGA2560.(OC0B)PG5
- new net PH4: ATMEGA2560.PH4(OC4B)
- new net PH5: ATMEGA2560.PH5(OC4C)
- new net PH6: ATMEGA2560.PH6(OC2B)
- new net PWRIN: D3.A, PWRIN_ON_LED.A, R54.1
- new net RESET: ATMEGA2560.RESET, C11.1, D4.A, ICSP.5, R11.2, RESET.3, RESET.4
- new net RI: ATMEGA2560.PJ3(PCINT12), FTDI.!RI
- new net RXD0: ATMEGA2560.(RXD0/PCIN8)PE0, FTDI.TXD
- new net RXD1: ATMEGA2560.(RXD1/INT2)PD2
- new net RXD2: ATMEGA2560.PH0(RXD2)
- new net RXD3: ATMEGA2560.PJ0(RXD3/PCINT9)
- new net RXL: FTDI.CBUS1, RX.C
- new net RX_1: U$1.DOUT
- new net SCK: ATMEGA2560.(SCK/PCINT1)PB1, ICSP.3, Q6.D, R47.1
- new net SCL: ATMEGA2560.(SCL/INT0)PD0, R13.2
- new net SDA: ATMEGA2560.(SDA/INT1)PD1, R12.2
- new net SD_CARD_DETECT_1: ATMEGA2560.PJ6(PCINT15), MICRO_SD_1.CD1
- new net SD_CS_HI: ATMEGA2560.PL1(ICP5), Q7.D, R49.1
- new net SD_CS_LO: MICRO_SD_1.!CS, Q7.S, R48.1
- new net SD_DI_LO: MICRO_SD_1.DI, Q4.S, R42.1
- new net SD_DO_LO: MICRO_SD_1.DO, Q5.S, R44.1
- new net SD_SCK_LO: MICRO_SD_1.SCK, Q6.S, R46.1
- new net SLEEP: ATMEGA2560.PJ2(XCK3/PCINT11), FTDI.CBUS4
- new net TXD0: ATMEGA2560.(TXD0)PE1, FTDI.RXD
- new net TXD1: ATMEGA2560.(TXD1/INT3)PD3
- new net TXD2: ATMEGA2560.PH1(TXD2)
- new net TXD3: ATMEGA2560.PJ1(TXD3/PCINT10)
- new net TXL: FTDI.CBUS0, TX.C
- new net TX_1: U$1.DIN
- new net USBVCC: C12.1, F1.1, T1.D, USB_POWER_ON_LED.A
- new net USHIELD: L1.2, USB_1.P$1, USB_1.P$2, Z1.1, Z2.1
- new net XBEE_SIGNAL_1: U$1.PWM0/RSSI
- new net XTAL1: ATMEGA2560.XTAL1, R5.1, Y1.3
- new net XTAL2: ATMEGA2560.XTAL2, R5.2, Y1.1
- new net XVCC: F1.2, USB_1.1
- net GND: now also C4.2, C5.2, LED2.C, U$1.GND
- net VIN: now also C8.1, D3.C, IC1.IN, PC1.+, R6.2
Other:
- note added: "(MISO)"
- note added: "(MOSI)"
- note added: "(RX0)"
- note added: "(SCK)"
- note added: "(TX0)"
- note added: "Arduino MEGA 2560"
- note added: "TM"
- note added: "pwm"
- moved on the sheet: B1, C1, C2, C3, D1, D2, FB1, JP1, LED1, R1, R2, R3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

Commit message: made it pretty with notes
Other:
- note added: "Arduino Mega Reference stuff"
- note added: "FTDI Chip for programming, needs reset logic still"
- note added: "GPS circuit from Adafruit"
- note added: "Micro SD slot and level shifting to make it work"
- note added: "Power stuff dfrom Arduino reference schematic, should change linear regulators to bucks probably for efficency"
- note added: "Random stuff, ICSP programing header, status leds, I2C pull ups"
- note added: "Reset Stuff"
- note added: "Xbee Reference Stuff"
- moved on the sheet: 3V3_ON_LED, 3V3_REV_LED, 5V_ON_LED, 5V_REV_LED, ATMEGA2560, B1, C1, C10, C11, C12, C13, C14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

Commit message: changed net names to fix errors
Connections:
- new net N$110: 5V_REV_LED.C, R37.2
- new net N$120: 3V3_ON_LED.C, R39.2
- net N$11: no longer 5V_REV_LED.C, R37.2
- net N$12: no longer 3V3_ON_LED.C, R39.2
Changed lines of the file:
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@@
 </segment>
 </net>
-<net name="N$11" class="0">
+<net name="N$110" class="0">
 <segment>
 <pinref part="5V_REV_LED" gate="G$1" pin="C"/>
@@
 </segment>
 </net>
-<net name="N$12" class="0">
+<net name="N$120" class="0">
 <segment>
 <pinref part="3V3_ON_LED" gate="G$1" pin="C"/>

Commit message: added bluetooth chip and condensed layout somewhat, still not routed
Parts:
- added C17, C18: 1uF, microbuilder:CAP_CERAMIC0805-NOOUTLINE
- added C19, C20: 10uF, microbuilder:CAP_CERAMIC0805-NOOUTLINE
- added D10, D11, D8, D9: 1n4148, microbuilder:DIODESOD-323
- added D12, D7: MBR120, microbuilder:DIODE-SCHOTTKYSOD-123
- added D5: RED, microbuilder:LED0805_NOOUTLINE
- added D6: GREEN, microbuilder:LED0805_NOOUTLINE
- added JP2: (no value), microbuilder:HEADER-1X876MIL
- added R14, R15: 1K, microbuilder:RESISTOR0805_NOOUTLINE
- added R16, R17: 100K, microbuilder:RESISTOR0805_NOOUTLINE
- added R18: 2K, microbuilder:RESISTOR0805_NOOUTLINE
- added SW1: EG1319, microbuilder:SWITCH_DPDTEG1390
- added TP1: SWCLK, microbuilder:TESTPOINT1.5X2.0MM_NOCREAM
- added TP2: SWDIO, microbuilder:TESTPOINT1.5X2.0MM_NOCREAM
- added TP3, VTREF: FCTRST, microbuilder:TESTPOINT1.5X2.0MM_NOCREAM
- added U$31, U$32: MOUNTINGHOLE2.5, microbuilder:MOUNTINGHOLE2.5
- added U3: (no value), microbuilder:NRF51822_MODULE_MDBT40
- added U4: MIC5225-3.3, microbuilder:VREG_SOT23-5
- added X1: JST 2PH, microbuilder:CON_JST_PH_2PIN
- added Y2: 32.768kHz (535-9166-2-ND), microbuilder:CRYSTAL2.0X6.0_32.768
Connections:
- new net CONNECTED_LED: R15.1, U3.P0.19
- new net CTS_3V: D8.A, R16.1, U3.P0.10
- new net CTS_5V: D8.C, JP2.7
- new net DFU_3V: D11.A, U3.P0.07
- new net DFU_5V: D11.C, JP2.1
- new net FCTRYRST_3V: TP3.P$1, U3.P0.16
- new net MODE_3V: D10.A, U3.P0.01/AIN2
- new net MODE_5V: D10.C, JP2.8, R18.1
- new net MODE_LED: R14.1, U3.P0.18
- new net N$15: D5.A, R14.2
- new net N$16: D6.A, R15.2
- new net N$17: U3.P0.26/AIN0/XL2, Y2.1
- new net N$18: U3.P0.27/AIN1/XL1, Y2.2
- new net N$19: R18.2, SW1.P2
- new net N$21: C19.1, D12.C, D7.C, U4.EN, U4.IN
- new net RTS_O: JP2.3, U3.P0.08
- new net RXD_3V: D9.A, R17.1, U3.P0.11
- new net RXD_5V: D9.C, JP2.5
- new net SWCLK: TP1.P$1, U3.SWCLK
- new net SWDIO/RST_3V: TP2.P$1, U3.SWDIO/NRESET
- new net TX_O: JP2.6, U3.P0.09
- new net VBAT: D7.A, X1.2
- net 3.3V: now also C17.1, C18.1, C20.1, R16.2, R17.2, SW1.O2, U3.AVDD, U3.VDD, U4.OUT, VTREF.P$1
- net GND: now also C17.2, C18.2, C19.2, C20.2, D5.C, D6.C, JP2.2, SW1.S2, U3.GND@1, U3.GND@2, U3.GND@3, U3.GND@4, U3.GND@5, U3.P0.30, U4.GND, X1.1
- net VIN: now also D12.A, JP2.4
Other:
- note added: "CMD"
- note added: "DATA"

Commit message: added flash chip and made text formal/pretty
Parts:
- removed MICRO_SD_1: MICRO-SD_CARD_SOCKET, SparkFun-Connectors:MICRO-SD_CARD_SOCKET
- removed Q4, Q5, Q6, Q7: 220mA/50V/3.5Ω, SparkFun-DiscreteSemi:MOSFET-NCH-BSS138
- removed R42, R43, R44, R45, R46, R47, R48, R49: (no value), rcl:R-US_M1206
- added C21: 10uF, microbuilder:CAP_CERAMIC_0805MP
- added JP3: (no value), microbuilder:HEADER-1X870MIL
- added R19, R20: 10K, microbuilder:RESISTOR_0805MP
- added U5: MB85RC256VPF-G-JNERE2, microbuilder:FRAM_SOIC8_I2C
Connections:
- removed net SD_CS_LO: MICRO_SD_1.!CS, Q7.S, R48.1
- removed net SD_DI_LO: MICRO_SD_1.DI, Q4.S, R42.1
- removed net SD_DO_LO: MICRO_SD_1.DO, Q5.S, R44.1
- removed net SD_SCK_LO: MICRO_SD_1.SCK, Q6.S, R46.1
- new net A0: JP3.1, U5.A0
- new net A1: JP3.2, U5.A1
- new net A2: JP3.3, U5.A2
- new net VCC: C21.1, JP3.8, R19.2, R20.2, U5.VCC
- new net WP: JP3.6, U5.WP
- net 3V3: no longer MICRO_SD_1.VCC, Q4.G, Q5.G, Q6.G, Q7.G, R42.2, R44.2, R46.2, R48.2
- net 5V: no longer R43.2, R45.2, R47.2, R49.2
- net 90348: no longer MICRO_SD_1.CD2, MICRO_SD_1.GND, MICRO_SD_1.SHIELD@1, MICRO_SD_1.SHIELD@3
- net GND: now also C21.2, JP3.7, U5.GND
- net MISO: no longer Q5.D, R45.1
- net MOSI: no longer Q4.D, R43.1
- net SCK: no longer Q6.D, R47.1
- net SCL: now also JP3.5, R19.1, U5.SCL
- net SDA: now also JP3.4, R20.1, U5.SDA
- net SD_CARD_DETECT_1: no longer MICRO_SD_1.CD1
- net SD_CS_HI: no longer Q7.D, R49.1
Other:
- note added: "Arduino Mega Reference"
- note added: "Bluetooth chip and relevant power circuitry from schematic"
- note added: "External Flash Chip"
- note added: "FTDI Chip for programming"
- note added: "I2C Address =1010 + A2 + A1 + A0"
- note added: "Misc circuitry, including ICSP programing header, status leds, I2C pull ups"
- note added: "Power circuitry dfrom Arduino reference schematic, may be changed from linear regulators to bucks for efficency"
- note added: "Reset"
- note added: "WP high = write protection enabled ... needs to go low to enable writing! (WP has internal pull-down)"
- note added: "Xbee Reference"
- note removed: "Arduino Mega Reference stuff"
- note removed: "FTDI Chip for programming, needs reset logic still"
- note removed: "Micro SD slot and level shifting to make it work"
- note removed: "Power stuff dfrom Arduino reference schematic, should change linear regulators to bucks probably for efficency"
- note removed: "Random stuff, ICSP programing header, status leds, I2C pull ups"
- note removed: "Reset Stuff"
- note removed: "Xbee Reference Stuff"
- moved on the sheet: C11, C17, C18, C19, C20, D10, D11, D12, D4, D5, D6, D7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

Commit message: unrouted, spaced out baoard
Parts:
- removed U$31, U$32: MOUNTINGHOLE2.5, microbuilder:MOUNTINGHOLE2.5
Changed lines of the file:
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@@
 <part name="TP1" library="microbuilder" deviceset="TESTPOINT" device="1.5X2.0MM_NOCREAM" value="SWCLK"/>
 <part name="TP2" library="microbuilder" deviceset="TESTPOINT" device="1.5X2.0MM_NOCREAM" value="SWDIO"/>
-<part name="U$31" library="microbuilder" deviceset="MOUNTINGHOLE" device="2.5"/>
-<part name="U$32" library="microbuilder" deviceset="MOUNTINGHOLE" device="2.5"/>
 <part name="U$33" library="microbuilder" deviceset="VIN" device=""/>
 <part name="TP3" library="microbuilder" deviceset="TESTPOINT" device="1.5X2.0MM_NOCREAM" value="FCTRST"/>
@@
 <attribute name="VALUE" x="-1279.652" y="-21.971" size="1.27" layer="95" align="center-left"/>
 </instance>
-<instance part="U$31" gate="G$1" x="-1216.66" y="-109.22" smashed="yes"/>
-<instance part="U$32" gate="G$1" x="-1221.74" y="-109.22" smashed="yes"/>
 <instance part="U$33" gate="G$1" x="-1399.54" y="-93.98" smashed="yes" rot="R90">
 <attribute name="VALUE" x="-1400.556" y="-95.504" size="1.27" layer="96" rot="R90"/>

Commit message: save before leaving for meeting
Changed lines of the file:
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@@
 <part name="IC7" library="linear" deviceset="LMV358?*" device="MM" technology="X" value="LMV358IDGKR"/>
 <part name="D4" library="diode" deviceset="DIODE-" device="MINIMELF" value="CD1206-S01575"/>
-<part name="LOGO1" library="logo" deviceset="ESD" device=""/>
 <part name="FTDI" library="ftdichip" deviceset="FT232R" device="L"/>
 <part name="FTDI_RESET" library="SparkFun-Connectors" deviceset="TEST-POINT" device="2"/>
@@
 <attribute name="VALUE" x="-1356.5886" y="-260.35" size="1.778" layer="96" rot="R90"/>
 </instance>
-<instance part="LOGO1" gate="G$1" x="-961.39" y="-25.4" smashed="yes"/>
 <instance part="FTDI" gate="1" x="-1060.45" y="-237.49" smashed="yes">
 <attribute name="NAME" x="-1070.61" y="-210.82" size="1.778" layer="95"/>
