File: BeaconBoard/beacon1.brd (EAGLE design)
At the start: 160 x 100 mm, 59 parts, among them CN1 BATT_IN_JST, CN4 LOAD_JST, IC1 NCP1117ST50T3G, IC7 LMV358IDGKR, Y1 CSTCE16M0V53-R0 16MHZ

Commit message: final board design
Parts:
- removed C8: 100n, SmartPrj:C1206K
- removed CN1: BATT_IN_JST, microbuilder:JSTPH2
- removed CN4: LOAD_JST, microbuilder:JSTPH2
- removed D3: M7, diode:SMB
- removed IC1: NCP1117ST50T3G, linear:SOT223
- removed JP2: (no value), microbuilder:1X08_ROUND_76
- removed PC1, PC2: 47u, rcl:PANASONIC_D
- added JP4, JP5: (no value), microbuilder:1X07_ROUND_70
- added JP6: (no value), microbuilder:1X08_ROUND_76
- added U1: M95M02-DWMN3TP/K, M95M02-DWMN3TP_K:SOIC127P600X175-8N
- JP3: device SparkFun:1X07 -> adafruit:1X08-BIG
- moved FTDI1 153.0 mm to (99.1, 54.6), flipped to the bottom, turned to 90 degrees
- moved JP3 136.9 mm to (81.3, 3.81), flipped to the bottom
- moved 3V3_REV_LED 133.8 mm to (63.5, 68.6)
- moved 5V_REV_LED1 133.8 mm to (69.8, 68.6)
- moved PWRIN_ON_LED 133.8 mm to (76.2, 68.6)
- moved PWRIN_REV_LED 133.8 mm to (83.8, 68.6)
- moved USB_POWER_ON_LED 133.8 mm to (92.7, 68.6)
- moved Y1 132.1 mm to (57.1, 76.2)
- moved 3V3_ON_LED 128.4 mm to (94.0, 31.8)
- moved 5V_ON_LED 128.4 mm to (81.3, 31.8)
- moved 5V_REV_LED 128.4 mm to (87.6, 31.8)
- moved L 128.4 mm to (76.2, 31.8)
- moved R4 128.4 mm to (69.8, 31.8)
- moved R10 127.9 mm to (69.8, 39.4)
- moved R11 127.9 mm to (64.8, 39.4)
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Connections:
- removed net +5V: 5V_REV_LED1.A, SOLAR.2
- removed net CD1: JP3.7
- removed net CS: JP3.1
- removed net CTS: FTDI1.2
- removed net DI: JP3.2
- removed net DO: JP3.6
- removed net N$8: JP2.5
- removed net RTSDTR: R1.2
- removed net RTS_O: JP2.3
- removed net SCK1: JP3.4
- removed net VCCOUT: FTDI1.3
- removed net VIN: C8.1, D3.C, IC1.3, JP1.2, JP2.4, PC1.+
- new net CD: JP3.8
- new net N$1: 5V_ON_LED1.A, JP10.2
- new net N$3: JP4.1, SOLAR.2
- new net PG: JP4.5
- new net PS: JP4.4
- net +5V2: no longer 5V_ON_LED1.A, CN1.2, CN4.2, JP10.2
- net 3.3V: now also JP3.2, JP5.5, U1.8; no longer JP3.3
- net 5.0V: now also 5V_REV_LED1.A, FTDI1.3, JP1.2, JP3.1, JP4.7, JP5.7, JP6.4
- net 5V: no longer IC1.2, IC1.4, PC2.+
- net 90348: no longer C8.2, IC1.1, ICSP.6, PC1.-, PC2.-
- net DFU_5V: now also JP6.1; no longer JP2.1
- net GND: now also ICSP.6, JP3.3, JP4.3, JP4.6, JP5.6, JP6.2, U1.4; no longer CN1.1, CN4.1, JP2.2, JP3.5
- net MISO: now also JP3.5, U1.2
- net MODE_5V: now also JP6.8; no longer JP2.8
- net MOSI: now also JP3.6, U1.5
- net PB0: now also JP3.7, U1.1
- net PB4: now also JP6.3
- net PB5: now also JP6.7
- net PB6: now also FTDI1.2
- net PWRIN: no longer D3.A
- net RESET: now also R1.2
- net RXD2: now also JP6.6; no longer JP2.6
- net SCK: now also JP3.4, U1.6
- net TXD2: now also JP6.5; no longer JP2.7
Routing:
- net 90348: track 0.00 -> 400.2 mm, vias 0 -> 14
- net GND: track 0.00 -> 359.1 mm
- net 5.0V: track 0.00 -> 319.9 mm
- net 5V: track 0.00 -> 214.2 mm, vias 0 -> 8
- net 3.3V: track 0.00 -> 197.4 mm, vias 0 -> 2
- net RESET: track 0.00 -> 175.7 mm, vias 0 -> 3
- net 3V3: track 0.00 -> 173.7 mm, vias 0 -> 2
- net N$110: track 0.00 -> 117.7 mm, vias 0 -> 2
- net N$26: track 0.00 -> 113.7 mm, vias 0 -> 3
- net PB5: track 0.00 -> 102.5 mm, vias 0 -> 2
- net MISO: track 0.00 -> 101.3 mm, vias 0 -> 2
- net SCK: track 0.00 -> 99.7 mm, vias 0 -> 1
- net MOSI: track 0.00 -> 95.0 mm, vias 0 -> 1
- net RXD3: track 0.00 -> 86.9 mm
- net TXD3: track 0.00 -> 83.0 mm
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Other:
- board size 160 x 100 mm -> 101.6 x 100 mm
