File: BeaconBoard/beacon1.sch (EAGLE design)
At the start: 108 parts, among them IC1 NCP1117ST50T3G, IC6 LP2985-33DBVR, IC7 LMV358IDGKR, SW1 EG1319, T1 FDN340P, U1 FGPMMOPA6H, U2 MIC5225-3.3, U4 MIC5225-3.3, U5 MB85RC256VPF-G-JNERE2, X1 JST 2PH, Y1 CSTCE16M0V53-R0 16MHZ, Y2 32.768kHz (535-9166-2-ND)

Commit message: i changed everything and only just comitted now cause im bad
Parts:
- removed B1: CR1220, microbuilder:BATTERYCR1220_SMT
- removed C1: 0.1uF, microbuilder:CAP_CERAMIC0805-NOOUTLINE
- removed C13: 1u, SmartPrj:C-EUC1206K
- removed C15, C16: 100n, SmartPrj:C-EUC1206K
- removed C17, C18: 1uF, microbuilder:CAP_CERAMIC0805-NOOUTLINE
- removed C19, C2, C20, C3: 10uF, microbuilder:CAP_CERAMIC0805-NOOUTLINE
- removed C21: 10uF, microbuilder:CAP_CERAMIC_0805MP
- removed D1: 1N4148, microbuilder:DIODESOD-323
- removed D10, D11, D8, D9: 1n4148, microbuilder:DIODESOD-323
- removed D12, D7: MBR120, microbuilder:DIODE-SCHOTTKYSOD-123
- removed D2: CUS520, microbuilder:DIODESOD-323
- removed D5: RED, microbuilder:LED0805_NOOUTLINE
- removed D6: GREEN, microbuilder:LED0805_NOOUTLINE
- removed FB1: Ferrite, microbuilder:FERRITE-0805NO
- removed IC6: LP2985-33DBVR, SmartPrj:LP2985-XXDBVR33
- removed LED1: RED, microbuilder:LED0805
- removed R1, R14, R15: 1K, microbuilder:RESISTOR0805_NOOUTLINE
- removed R16, R17: 100K, microbuilder:RESISTOR0805_NOOUTLINE
- removed R18: 2K, microbuilder:RESISTOR0805_NOOUTLINE
- removed R19, R20: 10K, microbuilder:RESISTOR_0805MP
- removed R2, R3: 10K, microbuilder:RESISTOR0805_NOOUTLINE
- removed R6, R7: 10k, adafruit:R-US_M1206
- removed SW1: EG1319, microbuilder:SWITCH_DPDTEG1390
- removed T1: FDN340P, zetex:PMOSSOT23
- removed TP1: SWCLK, microbuilder:TESTPOINT1.5X2.0MM_NOCREAM
- removed TP2: SWDIO, microbuilder:TESTPOINT1.5X2.0MM_NOCREAM
- removed TP3, VTREF: FCTRST, microbuilder:TESTPOINT1.5X2.0MM_NOCREAM
- removed U$20: U.FL, microbuilder:U.FL
- removed U1: FGPMMOPA6H, microbuilder:GPS_FGPMMOPA6H
- removed U2, U4: MIC5225-3.3, microbuilder:VREG_SOT23-5
- removed U3: (no value), microbuilder:NRF51822_MODULE_MDBT40
- removed X1: JST 2PH, microbuilder:CON_JST_PH_2PIN
- removed Y2: 32.768kHz (535-9166-2-ND), microbuilder:CRYSTAL2.0X6.0_32.768
- added 5V_ON_LED1: GREEN, SparkFun-LED:LED-GREENLILYPAD
- added 5V_REV_LED1: RED, SparkFun-LED:LED-RED1206
- added BATT1, BATT2: Battery, microbuilder:HEADER-1X2
- added C22, C23: 100m, SmartPrj:C-EUC1206K
- added CN1: BATT_IN_JST, microbuilder:JST_2PIN
- added CN4: LOAD_JST, microbuilder:JST_2PIN
- added JP10: LOAD_0.1, microbuilder:HEADER-1X2
- added JP11: BATT_IN_0.1, microbuilder:HEADER-1X2
- added JP8: PWR_IN_0.1, microbuilder:HEADER-1X2
- added SOLAR: Solar, microbuilder:HEADER-1X2
- added U$31: DC877A, DC877A:DC877A
- JP3: device microbuilder:HEADER-1X870MIL -> SparkFun:M07
- U5: value MB85RC256VPF-G-JNERE2 -> microSD; device microbuilder:FRAM_SOIC8_I2C -> SparkFun:USD-SOCKETSMD
Connections:
- removed net A0: JP3.1, U5.A0
- removed net A1: JP3.2, U5.A1
- removed net A2: JP3.3, U5.A2
- removed net CMP: C15.2, IC7B.+IN, R6.1, R7.2
- removed net CONNECTED_LED: R15.1, U3.P0.19
- removed net CTS_3V: D8.A, R16.1, U3.P0.10
- removed net DFU_3V: D11.A, U3.P0.07
- removed net FCTRYRST_3V: TP3.P$1, U3.P0.16
- removed net GATE_CMD: IC7B.OUT, T1.G
- removed net MODE_3V: D10.A, U3.P0.01/AIN2
- removed net MODE_LED: R14.1, U3.P0.18
- removed net N$1: B1.+, D2.A
- removed net N$15: D5.A, R14.2
- removed net N$16: D6.A, R15.2
- removed net N$17: U3.P0.26/AIN0/XL2, Y2.1
- removed net N$18: U3.P0.27/AIN1/XL1, Y2.2
- removed net N$19: R18.2, SW1.P2
- removed net N$2: LED1.C, R1.2
- removed net N$21: C19.1, D12.C, D7.C, U4.EN, U4.IN
- removed net N$3: FB1.P$1, U2.OUT
- removed net N$4: U$20.SIGNAL, U1.EX_ANT
- removed net RX: D1.C, JP1.4
- removed net RXD2: ATMEGA2560.PH0(RXD2)
- removed net RXD_3V: D9.A, R17.1, U3.P0.11
- removed net RX_3V: D1.A, R3.2, U1.RX
- removed net SWCLK: TP1.P$1, U3.SWCLK
- removed net SWDIO/RST_3V: TP2.P$1, U3.SWDIO/NRESET
- removed net TX: JP1.5, U1.TX
- removed net TXD2: ATMEGA2560.PH1(TXD2)
- removed net VBAT: D7.A, X1.2
- removed net VCC: C21.1, JP3.8, R19.2, R20.2, U5.VCC
- removed net WP: JP3.6, U5.WP
- new net +5V: 5V_REV_LED1.A, SOLAR.2
- new net +5V2: 5V_ON_LED1.A, BATT1.2, BATT2.2, CN1.2, CN4.2, JP10.2, JP11.2
- new net 5.0V: JP8.2
- new net CD1: JP3.7, U5.CD2
- new net CS: JP3.1, U5.CS
- new net DI: JP3.2, U5.DI
- new net DO: JP3.6, U5.DO
- new net GND2: BATT1.1
- new net GND3: BATT2.1
- new net N$22: C23.1, U$31.VOUT
- new net N$23: C22.1, U$31.VIN
- new net N$26: 5V_ON_LED1.C, 5V_REV_LED1.C, C22.2
- new net SCK1: JP3.4, U5.SCK
- net 1PPS: no longer U1.1PPS
- net 3.3V: now also C23.2, JP3.3, U5.VCC; no longer C1.1, C17.1, C18.1, C2.1, C20.1, FB1.P$2, R16.2, R17.2, R3.1, SW1.O2, U1.VCC, U3.AVDD, U3.VDD, U4.OUT, VTREF.P$1
- net 3V3: no longer C13.2, IC6.OUT, IC7B.-IN
- net 5V: no longer C16.2, IC6.IN, IC6.ON/!OFF, IC7P.V+, T1.S
- net 90348: now also U$31.GND; no longer C13.1, C15.1, C16.1, IC6.GND, IC7P.V-, R7.1
- net CTS_5V: no longer D8.C
- net DFU_5V: no longer D11.C
- net ENABLE: no longer R2.1, U2.EN
- net FIX: no longer LED1.A, U1.3D-FIX
- net GND: now also CN1.1, CN4.1, JP10.1, JP11.1, JP3.5, JP8.1, SOLAR.1, U5.SHIELD1, U5.SHIELD2; no longer B1.-, C1.2, C17.2, C18.2, C19.2, C2.2, C20.2, C21.2, C3.2, D5.C, D6.C, JP3.7, R1.1, SW1.S2, U$20.GND@0, U$20.GND@1, U1.GND@1, U1.GND@2, U1.GND@3, U1.GND@4, U2.GND, U3.GND@1, U3.GND@2, U3.GND@3, U3.GND@4, U3.GND@5, U3.P0.30, U4.GND, X1.1
- net MODE_5V: no longer D10.C, R18.1
- net RTS_O: no longer U3.P0.08
- net RXD0: now also JP1.5
- net RXD_5V: now also ATMEGA2560.PH1(TXD2); no longer D9.C
- net SCL: no longer JP3.5, R19.1, U5.SCL
- net SDA: no longer JP3.4, R20.1, U5.SDA
- net TXD0: now also JP1.4
- net TX_O: now also ATMEGA2560.PH0(RXD2); no longer U3.P0.09
- net USBVCC: no longer T1.D
- net VBACKUP: no longer D2.C, U1.VBACKUP
- net VIN: no longer C3.1, D12.A, R2.2, R6.2, U2.IN
Other:
- note added: "SD Card"
- note removed: "CMD"
- note removed: "D1+R3 restrict RX input to 3.3V"
- note removed: "DATA"
- note removed: "External Flash Chip"
- note removed: "I2C Address =1010 + A2 + A1 + A0"
- note removed: "WP high = write protection enabled ... needs to go low to enable writing! (WP has internal pull-down)"
- moved on the sheet: JP2

Commit message: removed full ftdi chip, reset board
Parts:
- removed C12, C14: 100n, SmartPrj:C-EUC1206K
- removed F1: MF-MSMF050-2 500mA, rcl:L-EUL1812
- removed FTDI: FT232RL, ftdichip:FT232RL
- removed FTDI_RESET: TEST-POINT2, SparkFun-Connectors:TEST-POINT2
- removed L1: BLM21, wuerth-elektronik:WE-CBF_0805
- removed R8, R9: 1k, adafruit:R-US_M1206
- removed RX, TX: YELLOW, led:LEDSMT1206
- removed U5: microSD, SparkFun:USD-SOCKETSMD
- removed USB_1: USB-B_TH, SmartPrj:PN61729
- removed Z1, Z2: CG0603MLC-05E, varistor:VARISTORCN0603
- added FTDI1: (no value), adafruit:PINHD-1X6CB
- added R1: 10, adafruit:R-US_R0805
Connections:
- net TX_O renamed RXD2
- removed net CTS_5V: JP2.7
- removed net D+: FTDI.USBDP, USB_1.3, Z2.2
- removed net D-: FTDI.USBDM, USB_1.2, Z1.2
- removed net N$11: FTDI.CBUS2
- removed net N$12: FTDI.CBUS3
- removed net N$54: R9.1, RX.A
- removed net N$55: R8.1, TX.A
- removed net N$9: FTDI.!RESET, FTDI_RESET.1
- removed net RXD_5V: ATMEGA2560.PH1(TXD2), JP2.5
- removed net RXL: FTDI.CBUS1, RX.C
- removed net TXL: FTDI.CBUS0, TX.C
- removed net USHIELD: L1.2, USB_1.P$1, USB_1.P$2, Z1.1, Z2.1
- removed net XVCC: F1.2, USB_1.1
- new net CTS: FTDI1.2
- new net N$2: FTDI1.6, R1.1
- new net RTSDTR: R1.2
- new net TXD2: ATMEGA2560.PH1(TXD2), JP2.7
- new net VCCOUT: FTDI1.3
- net 3.3V: no longer U5.VCC
- net 5V: no longer C14.1, FTDI.VCC, FTDI.VCCIO, R8.2, R9.2
- net 90348: no longer C12.2, C14.2, FTDI.GND@1, FTDI.GND@A, L1.1, USB_1.4
- net CD1: no longer U5.CD2
- net CS: no longer U5.CS
- net DI: no longer U5.DI
- net DO: no longer U5.DO
- net GND: now also FTDI1.1; no longer U5.GND, U5.SHIELD1, U5.SHIELD2
- net N$8: now also JP2.5; no longer FTDI.GND, FTDI.GND@2, FTDI.TEST
- net RI: no longer FTDI.!RI
- net RXD0: now also FTDI1.4; no longer ATMEGA2560.(RXD0/PCIN8)PE0, FTDI.TXD, JP1.5
- net RXD3: now also JP1.5
- net SCK1: no longer U5.SCK
- net SLEEP: no longer FTDI.CBUS4
- net TXD0: now also FTDI1.5; no longer ATMEGA2560.(TXD0)PE1, FTDI.RXD, JP1.4
- net TXD3: now also JP1.4
- net USBVCC: no longer C12.1, F1.1
Other:
- note removed: "(RX0)"
- note removed: "(TX0)"

Commit message: final board design
Parts:
- removed C8: 100n, SmartPrj:C-EUC1206K
- removed CN1: BATT_IN_JST, microbuilder:JST_2PIN
- removed CN4: LOAD_JST, microbuilder:JST_2PIN
- removed D3: M7, diode:DIODE-SMB
- removed IC1: NCP1117ST50T3G, linear:MC33269ST-3.3T3
- removed JP2: (no value), microbuilder:HEADER-1X876MIL
- removed PC1, PC2: 47u, rcl:CPOL-EUD
- added JP4, JP5: (no value), microbuilder:HEADER-1X770MIL
- added JP6: (no value), microbuilder:HEADER-1X876MIL
- added U1: M95M02-DWMN3TP/K, M95M02-DWMN3TP_K:M95M02-DWMN3TP/K
- JP3: device SparkFun:M07 -> adafruit:PINHD-1X8BIG
Connections:
- removed net +5V: 5V_REV_LED1.A, SOLAR.2
- removed net CD1: JP3.7
- removed net CS: JP3.1
- removed net CTS: FTDI1.2
- removed net DI: JP3.2
- removed net DO: JP3.6
- removed net N$8: JP2.5
- removed net RTSDTR: R1.2
- removed net RTS_O: JP2.3
- removed net SCK1: JP3.4
- removed net VCCOUT: FTDI1.3
- removed net VIN: C8.1, D3.C, IC1.IN, JP1.2, JP2.4, PC1.+
- new net CD: JP3.8
- new net N$1: 5V_ON_LED1.A, JP10.2
- new net N$3: JP4.1, SOLAR.2
- new net PG: JP4.5
- new net PS: JP4.4
- net +5V2: no longer 5V_ON_LED1.A, CN1.2, CN4.2, JP10.2
- net 3.3V: now also JP3.2, JP5.5, U1.VCC; no longer JP3.3
- net 5.0V: now also 5V_REV_LED1.A, FTDI1.3, JP1.2, JP3.1, JP4.7, JP5.7, JP6.4
- net 5V: no longer IC1.OUT, IC1.OUT@1, PC2.+
- net 90348: no longer C8.2, IC1.GND/ADJ, ICSP.6, PC1.-, PC2.-
- net DFU_5V: now also JP6.1; no longer JP2.1
- net GND: now also ICSP.6, JP3.3, JP4.3, JP4.6, JP5.6, JP6.2, U1.VSS; no longer CN1.1, CN4.1, JP2.2, JP3.5
- net MISO: now also JP3.5, U1.Q
- net MODE_5V: now also JP6.8; no longer JP2.8
- net MOSI: now also JP3.6, U1.D
- net PB0: now also JP3.7, U1.!S
- net PB4: now also JP6.3
- net PB5: now also JP6.7
- net PB6: now also FTDI1.2
- net PWRIN: no longer D3.A
- net RESET: now also R1.2
- net RXD2: now also JP6.6; no longer JP2.6
- net SCK: now also JP3.4, U1.C
- net TXD2: now also JP6.5; no longer JP2.7
Other:
- note added: "SD Card and EEPROM"
- note removed: "SD Card"
- moved on the sheet: BATT1, BATT2, JP11, SOLAR
