File: BeaconBoard2/PCBFORNICOLESAVE.brd (EAGLE design)
At the start: 101.6 x 101.6 mm, 108 parts, among them Q1 FDC645N, U1 ATMega2560, U2 3X3BGA0.4MM

Commit message: removed GPS pps line
Parts:
- moved R2 0.63 mm to (-15.2, -30.5)
- turned D1 to 90 degrees
Routing:
- net SD_3V3: track 0.00 -> 24.5 mm
- net 3V3: track 271.8 -> 284.9 mm, vias 11 -> 13
- net N$1: track 0.00 -> 3.38 mm
- removed copper zone on layer 1, net SD_GND
Changed lines of the file:
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@@
 <attribute name="VALUE" x="-13.24" y="-34.29" size="0.8128" layer="27" rot="R90" align="center"/>
 </element>
-<element name="R2" library="Resistors" package="0603" value="10k" x="-15.24" y="-31.115" smashed="yes" rot="R180">
-<attribute name="NAME" x="-15.24" y="-32.385" size="1.016" layer="25" rot="R180" align="center"/>
-<attribute name="VALUE" x="-15.24" y="-29.845" size="1.016" layer="27" rot="R180" align="center"/>
-</element>
-<element name="D1" library="Diodes" package="1206" value="" x="-11.43" y="-33.02" smashed="yes" rot="R270">
-<attribute name="NAME" x="-9.906" y="-33.02" size="0.8128" layer="25" rot="R270" align="center"/>
+<element name="R2" library="Resistors" package="0603" value="10k" x="-15.24" y="-30.48" smashed="yes" rot="R180">
+<attribute name="NAME" x="-15.24" y="-31.75" size="1.016" layer="25" rot="R180" align="center"/>
+<attribute name="VALUE" x="-15.24" y="-29.21" size="1.016" layer="27" rot="R180" align="center"/>
+</element>
+<element name="D1" library="Diodes" package="1206" value="" x="-11.43" y="-33.02" smashed="yes" rot="R90">
+<attribute name="NAME" x="-12.954" y="-33.02" size="0.8128" layer="25" rot="R90" align="center"/>
 </element>
 <element name="D2" library="Diodes" package="1206" value="" x="-8.89" y="-33.02" smashed="yes" rot="R270">
@@
 <wire x1="12.065" y1="-35.71875" x2="13.97" y2="-35.71875" width="0.8128" layer="1"/>
 <wire x1="13.97" y1="-35.71875" x2="13.97" y2="-35.712" width="0.8128" layer="1"/>
-<wire x1="0.3" y1="-25.57625" x2="-2.12725" y2="-28.0035" width="0.6096" layer="1"/>
-<wire x1="-2.12725" y1="-28.0035" x2="-8.89" y2="-28.0035" width="0.6096" layer="1"/>
 <wire x1="-15.5575" y1="-28.0035" x2="-15.621" y2="-27.94" width="0.6096" layer="1"/>
 <wire x1="35.96" y1="-20.44" x2="35.96" y2="-18.561" width="0.8128" layer="1"/>
@@
 <contactref element="Q1" pad="6"/>
 <contactref element="Q1" pad="PAD"/>
+<wire x1="-15.621" y1="-27.94" x2="-8.9535" y2="-27.94" width="0.254" layer="1"/>
+<wire x1="-8.9535" y1="-27.94" x2="-8.89" y2="-28.0035" width="0.254" layer="1"/>
+<wire x1="-5.21" y1="-13.0175" x2="-5.21" y2="-16.64" width="0.254" layer="1"/>
+<wire x1="-5.21" y1="-16.64" x2="-7.62" y2="-19.05" width="0.254" layer="1"/>
+<via x="-7.62" y="-19.05" extent="1-16" drill="0.35"/>
+<wire x1="-7.62" y1="-19.05" x2="-8.89" y2="-20.32" width="0.254" layer="16"/>
+<wire x1="-8.89" y1="-20.32" x2="-8.89" y2="-25.4" width="0.254" layer="16"/>
+<via x="-8.89" y="-25.4" extent="1-16" drill="0.35"/>
+<wire x1="-8.89" y1="-25.4" x2="-8.89" y2="-28.0035" width="0.254" layer="1"/>
 <wire x1="14.2875" y1="30.00375" x2="18.85" y2="35.56" width="0" layer="19" extent="1-1"/>
 <wire x1="13.465" y1="28.2575" x2="13.335" y2="29.05125" width="0" layer="19" extent="1-16"/>
@@
 <wire x1="6.0325" y1="-5.3975" x2="6.0325" y2="-1" width="0" layer="19" extent="1-16"/>
 <wire x1="-3.5" y1="-6.0325" x2="0" y2="0" width="0" layer="19" extent="1-16"/>
-<wire x1="0.3" y1="-25.57625" x2="-5.21" y2="-13.0175" width="0" layer="19" extent="1-1"/>
-<wire x1="-15.5575" y1="-28.0035" x2="-8.89" y2="-28.0035" width="0" layer="19" extent="1-1"/>
 <wire x1="-16.155" y1="-34.29" x2="-15.5575" y2="-28.0035" width="0" layer="19" extent="1-1"/>
 <wire x1="-16.155" y1="-34.94" x2="-16.155" y2="-34.29" width="0" layer="19" extent="1-1"/>
@@
 <wire x1="-28.829" y1="11.43" x2="-22.86" y2="1.27" width="0" layer="19" extent="1-1"/>
 <wire x1="-31.75" y1="11.43" x2="-28.829" y2="11.43" width="0" layer="19" extent="1-1"/>
-<wire x1="-16.129" y1="-31.115" x2="-6.5" y2="-23.945" width="0" layer="19" extent="1-1"/>
-<wire x1="-17.4625" y1="-33.02" x2="-16.129" y2="-31.115" width="0" layer="19" extent="1-1"/>
+<wire x1="-16.129" y1="-30.48" x2="-6.5" y2="-23.945" width="0" layer="19" extent="1-1"/>
+<wire x1="-17.4625" y1="-33.02" x2="-16.129" y2="-30.48" width="0" layer="19" extent="1-1"/>
 <wire x1="-24.257" y1="-27.94" x2="-17.4625" y2="-33.02" width="0" layer="19" extent="1-1"/>
 <wire x1="-28.5" y1="-29.5" x2="-24.257" y2="-27.94" width="0" layer="19" extent="1-1"/>
@@
 <wire x1="23.96" y1="-35.44" x2="34.46" y2="-35.44" width="0" layer="19" extent="1-1"/>
 <wire x1="19.05" y1="-35.712" x2="23.96" y2="-35.44" width="0" layer="19" extent="1-1"/>
-<wire x1="-4.7" y1="-36.445" x2="-16.129" y2="-31.115" width="0" layer="19" extent="1-1"/>
+<wire x1="-4.7" y1="-36.445" x2="-16.129" y2="-30.48" width="0" layer="19" extent="1-1"/>
 <wire x1="3.3" y1="-36.345" x2="-4.7" y2="-36.445" width="0" layer="19" extent="1-1"/>
 </signal>
@@
 </signal>
 <signal name="SD_GND">
-<polygon width="0.3048" layer="1" spacing="0.254" rank="5">
-<vertex x="-17.78" y="-38.1"/>
-<vertex x="7.9375" y="-38.1"/>
-<vertex x="7.9375" y="-22.86"/>
-<vertex x="-12.7" y="-22.86"/>
-<vertex x="-12.7" y="-32.385"/>
-<vertex x="-14.605" y="-34.29"/>
-<vertex x="-17.78" y="-34.29"/>
-</polygon>
 <via x="-6.35" y="-26.67" extent="1-16" drill="0.381"/>
 <wire x1="-6.35" y1="-26.67" x2="-6.35" y2="-34.925" width="0.6096" layer="16"/>
@@
 <contactref element="D1" pad="2"/>
 <contactref element="R2" pad="1"/>
-<wire x1="-14.351" y1="-31.115" x2="-11.43" y2="-34.442" width="0" layer="19" extent="1-1"/>
+<wire x1="-14.351" y1="-30.48" x2="-12.548" y2="-30.48" width="0.254" layer="1"/>
+<wire x1="-12.548" y1="-30.48" x2="-11.43" y2="-31.598" width="0.254" layer="1"/>
 </signal>
 <signal name="SD_3V3">
@@
 <contactref element="Q1" pad="S"/>
 <contactref element="D1" pad="1"/>
-<wire x1="-15.24" y1="-33.64" x2="-16.155" y2="-33.64" width="0" layer="19" extent="1-1"/>
-<wire x1="-11.43" y1="-31.598" x2="-15.24" y2="-33.64" width="0" layer="19" extent="1-1"/>
-<wire x1="0.3" y1="-23.645" x2="-11.43" y2="-31.598" width="0" layer="19" extent="1-1"/>
+<wire x1="-15.24" y1="-33.64" x2="-16.155" y2="-33.64" width="0.254" layer="1"/>
+<wire x1="-15.09395" y1="-32.1167125" x2="-14.7145375" y2="-31.7373" width="0.254" layer="1"/>
+<wire x1="-15.24" y1="-33.64" x2="-15.09395" y2="-33.49395" width="0.254" layer="1"/>
+<wire x1="-15.09395" y1="-33.49395" x2="-15.09395" y2="-32.1167125" width="0.254" layer="1"/>
+<wire x1="-14.7145375" y1="-31.7373" x2="-14.1347" y2="-31.7373" width="0.254" layer="1"/>
+<wire x1="-14.1347" y1="-31.7373" x2="-11.43" y2="-34.442" width="0.254" layer="1"/>
+<wire x1="-11.43" y1="-34.442" x2="-10.497" y2="-34.442" width="0.254" layer="1"/>
+<wire x1="-10.497" y1="-34.442" x2="-10.0963" y2="-34.0413" width="0.254" layer="1"/>
+<wire x1="-10.0963" y1="-34.0413" x2="-10.0963" y2="-33.51575" width="0.254" layer="1"/>
+<wire x1="-0.1452" y1="-24.0902" x2="0.3" y2="-23.645" width="0.254" layer="1"/>
+<wire x1="-10.0963" y1="-33.51575" x2="-9.28335" y2="-32.7028" width="0.254" layer="1"/>
+<wire x1="-9.28335" y1="-32.7028" x2="-7.86225" y2="-32.7028" width="0.254" layer="1"/>
+<wire x1="-7.86225" y1="-32.7028" x2="-0.1452" y2="-24.98575" width="0.254" layer="1"/>
+<wire x1="-0.1452" y1="-24.98575" x2="-0.1452" y2="-24.0902" width="0.254" layer="1"/>
 </signal>
 </signals>

Commit message: removed sd_gnd traces
Routing:
- net SD_GND: track 8.25 -> 0.00 mm, vias 2 -> 0
Changed lines of the file:
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@@
 <wire x1="-0.9525" y1="-11.43" x2="-0.9525" y2="-10.795" width="0.3048" layer="1"/>
 <wire x1="-8" y1="1" x2="-9.89" y2="1" width="0.3048" layer="1"/>
-<wire x1="-9.89" y1="1" x2="-10.16" y2="1.27" width="0.3048" layer="1"/>
+<wire x1="-10.16" y1="1.27" x2="-9.89" y2="1" width="0.3048" layer="1"/>
 <contactref element="R15" pad="2"/>
 <contactref element="C27" pad="2"/>
@@
 <wire x1="-8.89" y1="-29.7815" x2="-8.89" y2="-31.598" width="0.3048" layer="1"/>
 </signal>
-<signal name="SD_GND">
-<via x="-6.35" y="-26.67" extent="1-16" drill="0.381"/>
-<wire x1="-6.35" y1="-26.67" x2="-6.35" y2="-34.925" width="0.6096" layer="16"/>
-<via x="-6.35" y="-34.925" extent="1-16" drill="0.381"/>
-</signal>
 <signal name="SOLAR+">

Commit message: removed GPS pps (again)
Parts:
- removed GPS_PPS, GPS_RX: JUMPER30V, Connectors:JUMPER_30V
- added R3: 1k, Resistors:0603
- moved R2 0.63 mm to (-15.2, -31.1)
- turned D1 to 270 degrees
Connections:
- removed net GPS_FLEX: GPS_PPS.1, GPS_RX.2, R31.2, U1.46
- removed net GPS_PPS: GPS.P$13, GPS_PPS.2
- removed net SD_3V3: D1.1, Q1.4, Q1.S, SD.4
- new net SD_GND: D1.2, Q1.1, Q1.2, Q1.5, Q1.6, Q1.PAD, SD.1, SD.6, SD.8, SD.S0, SD.S1, SD.S2, SD.S3
- net 3V3: now also R3.1, SD.4; no longer Q1.1, Q1.2, Q1.5, Q1.6, Q1.PAD
- net GND: now also Q1.4, Q1.S; no longer SD.1, SD.6, SD.8, SD.S0, SD.S1, SD.S2, SD.S3
- net GPS_RX: now also R31.2, U1.46; no longer GPS_RX.1
- net N$1: now also D1.1, R3.2; no longer D1.2, R2.1
- net SD_PWR: now also R2.1
Routing:
- net GPS_RX: track 6.59 -> 37.0 mm
- net GPS_FLEX: track 29.8 -> 0.00 mm
- net SD_3V3: track 24.5 -> 0.00 mm
- net 3V3: track 284.9 -> 298.1 mm, vias 13 -> 12
- net SD_GND: track 0.00 -> 11.7 mm, vias 0 -> 2
- net GPS_PPS: track 9.73 -> 0.00 mm
- net N$1: track 3.38 -> 1.82 mm
- net SD_PWR: track 32.9 -> 34.0 mm
- added copper zone on layer 1, net SD_GND

Commit message: finished routing, fixed DRC errors and wire stubs, moved components to make soldering easier
Parts:
- removed D1: (no value), Diodes:1206
- removed Q1: FDC645N, Transistors:WDFN-6
- removed R3: 1k, Resistors:0603
- added Q3: FDN340P, FDN340P:SSOT-3
- moved C26 1.90 mm to (-11.7, 27.9)
- moved Y1 1.42 mm to (0.32, -11.4)
- moved L1 1.27 mm to (11.4, 35.2)
- moved C17 1.27 mm to (-3.81, -14.3)
- moved C25 1.27 mm to (-14.6, 27.9)
- moved R2 1.27 mm to (-14.0, -31.1)
- moved R29 1.27 mm to (-19.1, 14.0)
- moved R30 1.27 mm to (-19.1, 16.5)
- moved L2 1.27 mm to (-21.0, 33.3)
- moved R26 0.90 mm to (-29.5, 4.45)
- moved C7 0.90 mm to (10.8, -8.10)
- moved C24 0.64 mm to (-17.1, 27.9)
- moved R27 0.64 mm to (14.0, -29.8)
- moved R28 0.64 mm to (-29.5, 1.27)
- moved R31 0.64 mm to (16.5, -29.8)
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Connections:
- removed net SD_GND: D1.2, Q1.1, Q1.2, Q1.5, Q1.6, Q1.PAD, SD.1, SD.6, SD.8, SD.S0, SD.S1, SD.S2, SD.S3
- new net SD_3V3: SD.4
- net 3V3: now also Q3.3; no longer R3.1, SD.4
- net GND: now also SD.1, SD.6, SD.8, SD.S0, SD.S1, SD.S2, SD.S3; no longer Q1.4, Q1.S
- net N$1: now also Q3.2, R2.1; no longer D1.1, R3.2
- net SD_PWR: now also Q3.1; no longer Q1.3, R2.1
Routing:
- net SD_GND: track 11.7 -> 0.00 mm, vias 2 -> 0
- net PA2: track 39.3 -> 32.4 mm
- net PA1: track 41.9 -> 35.5 mm
- net PA0: track 44.6 -> 38.3 mm
- net PA3: track 35.7 -> 30.2 mm
- net PA4: track 33.9 -> 29.3 mm
- net PA5: track 32.1 -> 28.5 mm
- net RESET: track 87.3 -> 90.7 mm
- net PA6: track 30.4 -> 27.6 mm
- net GND: track 18.3 -> 15.8 mm
- net BATT+: track 18.6 -> 21.0 mm
- net N$1: track 1.82 -> 3.93 mm
- net XTAL1: track 4.47 -> 6.37 mm
- net PA7: track 28.6 -> 26.8 mm
- net SD_PWR: track 34.0 -> 35.7 mm
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- removed copper zone on layer 1, net SD_GND

Commit message: rerouted sd card slightly to fix mistake
Parts:
- removed R2: 10k, Resistors:0603
Connections:
- removed net N$1: Q3.2, R2.1
- net GND: no longer R2.2
- net SD_3V3: now also Q3.2
Routing:
- net SD_3V3: track 0.00 -> 20.8 mm
- net GND: track 15.8 -> 26.4 mm, vias 21 -> 23
- net N$1: track 3.93 -> 0.00 mm
Changed lines of the file:
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@@
 </element>
 <element name="SD" library="Connectors" package="USD,FRONT" value="MICROSDFRONT" x="0" y="-29.845" smashed="yes" rot="R180"/>
-<element name="R2" library="Resistors" package="0603" value="10k" x="-13.97" y="-31.115" smashed="yes" rot="R180">
-<attribute name="NAME" x="-13.97" y="-32.385" size="1.016" layer="25" rot="R180" align="center"/>
-<attribute name="VALUE" x="-13.97" y="-29.845" size="1.016" layer="27" rot="R180" align="center"/>
-</element>
 <element name="D2" library="Diodes" package="1206" value="" x="-8.89" y="-33.02" smashed="yes" rot="R270">
 <attribute name="NAME" x="-7.366" y="-33.02" size="0.8128" layer="25" rot="R270" align="center"/>
@@
 <contactref element="SD" pad="S1"/>
 <contactref element="SD" pad="6"/>
-<contactref element="R2" pad="2"/>
 <wire x1="-10.16" y1="1.3335" x2="-9.8265" y2="1" width="0.254" layer="1"/>
 <wire x1="-9.8265" y1="1" x2="-8" y2="1" width="0.254" layer="1"/>
 <wire x1="11.43" y1="32.15" x2="11.43" y2="33.17875" width="0.254" layer="1"/>
+<wire x1="2.54" y1="-23.685" x2="2.5" y2="-23.645" width="0.254" layer="1"/>
+<wire x1="-3" y1="-23.645" x2="-3.175" y2="-23.82" width="0.254" layer="1"/>
+<wire x1="-3.175" y1="-23.82" x2="-3.175" y2="-26.035" width="0.254" layer="1"/>
+<via x="-3.175" y="-26.035" extent="1-16" drill="0.35"/>
+<wire x1="2.5" y1="-23.645" x2="2.5" y2="-25.995" width="0.254" layer="1"/>
+<wire x1="2.5" y1="-25.995" x2="2.54" y2="-26.035" width="0.254" layer="1"/>
+<via x="2.54" y="-26.035" extent="1-16" drill="0.35"/>
+<wire x1="-3.175" y1="-26.035" x2="2.54" y2="-26.035" width="0.254" layer="16"/>
 </signal>
 <signal name="BT_TX">
@@
 <wire x1="-10.795" y1="-13.17625" x2="-10.31875" y2="-13.6525" width="0.3048" layer="1"/>
 <via x="-10.31875" y="-13.6525" extent="1-16" drill="0.381"/>
-<wire x1="-10.31875" y1="-13.6525" x2="-3.478696875" y2="-20.492553125" width="0.3048" layer="16"/>
-<wire x1="-3.478696875" y1="-20.492553125" x2="-3.33375" y2="-33.9725" width="0.3048" layer="16"/>
+<wire x1="-10.31875" y1="-13.6525" x2="-4.7625" y2="-19.20875" width="0.3048" layer="16"/>
+<wire x1="-4.617553125" y1="-32.688696875" x2="-3.33375" y2="-33.9725" width="0.3048" layer="16"/>
+<wire x1="-4.617553125" y1="-32.688696875" x2="-4.7625" y2="-19.20875" width="0.3048" layer="16"/>
 </signal>
 <signal name="DBG_RX">
@@
 <signal name="SD_3V3">
 <contactref element="SD" pad="4"/>
-</signal>
-<signal name="N$1">
 <contactref element="Q3" pad="2"/>
-<contactref element="R2" pad="1"/>
-<wire x1="-14.14" y1="-34.61" x2="-13.26" y2="-33.73" width="0.254" layer="1"/>
-<wire x1="-13.26" y1="-33.73" x2="-13.081" y2="-33.551" width="0.254" layer="1"/>
-<wire x1="-13.081" y1="-33.551" x2="-13.081" y2="-31.115" width="0.254" layer="1"/>
+<wire x1="-9.52425" y1="-28.3972" x2="-2.9972" y2="-28.3972" width="0.254" layer="1"/>
+<wire x1="-9.7028" y1="-28.57575" x2="-9.52425" y2="-28.3972" width="0.254" layer="1"/>
+<wire x1="-14.14" y1="-34.61" x2="-9.7028" y2="-30.1728" width="0.254" layer="1"/>
+<wire x1="-9.7028" y1="-30.1728" x2="-9.7028" y2="-28.57575" width="0.254" layer="1"/>
+<wire x1="-2.9972" y1="-28.3972" x2="0.3" y2="-25.1" width="0.254" layer="1"/>
+<wire x1="0.3" y1="-25.1" x2="0.3" y2="-23.645" width="0.254" layer="1"/>
 </signal>
 </signals>

Commit message: fixed sd card mosfet
Parts:
- added D1: (no value), Diodes:1206
- added R2: 1k, Resistors:0603
- moved Q3 5.24 mm to (-14.0, -30.5)
Connections:
- new net N$1: D1.2, R2.2
- net GND: now also R2.1
- net SD_3V3: now also D1.1
Routing:
- net N$1: track 0.00 -> 14.5 mm
- net GND: track 26.4 -> 34.1 mm
- net 3V3: track 298.5 -> 293.3 mm
- net SD_3V3: track 20.8 -> 24.6 mm
- net SD_PWR: track 35.7 -> 34.3 mm
Changed lines of the file:
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@@
 <attribute name="VALUE" x="-23.495" y="31.75" size="1.27" layer="27" rot="R90"/>
 </element>
-<element name="Q3" library="FDN340P" package="SSOT-3" value="FDN340P" x="-15.24" y="-35.56" smashed="yes" rot="R90">
-<attribute name="AVAILABILITY" value="Unavailable" x="-15.24" y="-35.56" size="1.778" layer="27" rot="R90" display="off"/>
-<attribute name="DESCRIPTION" value=" Die Assymertrical For Fdc6329l " x="-15.24" y="-35.56" size="1.778" layer="27" rot="R90" display="off"/>
-<attribute name="MF" value="MICROSS/On Semiconductor" x="-15.24" y="-35.56" size="1.778" layer="27" rot="R90" display="off"/>
-<attribute name="MP" value="FDN340P" x="-15.24" y="-35.56" size="1.778" layer="27" rot="R90" display="off"/>
-<attribute name="NAME" x="-16.510309375" y="-34.289690625" size="1.016240625" layer="25" ratio="18" rot="R90"/>
-<attribute name="PACKAGE" value="TO-236-3 Micross" x="-15.24" y="-35.56" size="1.778" layer="27" rot="R90" display="off"/>
-<attribute name="PRICE" value="None" x="-15.24" y="-35.56" size="1.778" layer="27" rot="R90" display="off"/>
-<attribute name="VALUE" x="-12.058709375" y="-37.46876875" size="0.814409375" layer="27" ratio="10" rot="R90"/>
+<element name="Q3" library="FDN340P" package="SSOT-3" value="FDN340P" x="-13.97" y="-30.48" smashed="yes" rot="R90">
+<attribute name="AVAILABILITY" value="Unavailable" x="-13.97" y="-30.48" size="1.778" layer="27" rot="R90" display="off"/>
+<attribute name="DESCRIPTION" value=" Die Assymertrical For Fdc6329l " x="-13.97" y="-30.48" size="1.778" layer="27" rot="R90" display="off"/>
+<attribute name="MF" value="MICROSS/On Semiconductor" x="-13.97" y="-30.48" size="1.778" layer="27" rot="R90" display="off"/>
+<attribute name="MP" value="FDN340P" x="-13.97" y="-30.48" size="1.778" layer="27" rot="R90" display="off"/>
+<attribute name="NAME" x="-15.240309375" y="-29.209690625" size="1.016240625" layer="25" ratio="18" rot="R90"/>
+<attribute name="PACKAGE" value="TO-236-3 Micross" x="-13.97" y="-30.48" size="1.778" layer="27" rot="R90" display="off"/>
+<attribute name="PRICE" value="None" x="-13.97" y="-30.48" size="1.778" layer="27" rot="R90" display="off"/>
+<attribute name="VALUE" x="-10.788709375" y="-32.38876875" size="0.814409375" layer="27" ratio="10" rot="R90"/>
+</element>
+<element name="D1" library="Diodes" package="1206" value="" x="-15.24" y="-35.56" smashed="yes" rot="R180">
+<attribute name="NAME" x="-15.24" y="-37.084" size="0.8128" layer="25" rot="R180" align="center"/>
+</element>
+<element name="R2" library="Resistors" package="0603" value="1k" x="-31.75" y="-36.195" smashed="yes">
+<attribute name="NAME" x="-31.75" y="-34.925" size="1.016" layer="25" align="center"/>
+<attribute name="VALUE" x="-31.75" y="-37.465" size="1.016" layer="27" align="center"/>
 </element>
 </elements>
@@
 <wire x1="-5.21" y1="-14.2875" x2="-8.7025" y2="-17.78" width="0.254" layer="1"/>
 <wire x1="-8.89" y1="-17.78" x2="-8.7025" y2="-17.78" width="0.254" layer="1"/>
-<wire x1="-16.34" y1="-30.31" x2="-16.34" y2="-35.56" width="0.254" layer="1"/>
-<wire x1="-15.621" y1="-29.591" x2="-16.34" y2="-30.31" width="0.254" layer="1"/>
-<wire x1="-15.621" y1="-29.591" x2="-15.621" y2="-27.94" width="0.254" layer="1"/>
+<wire x1="-15.621" y1="-27.94" x2="-15.621" y2="-29.929" width="0.254" layer="1"/>
+<wire x1="-15.07" y1="-30.48" x2="-15.621" y2="-29.929" width="0.254" layer="1"/>
 <wire x1="-15.621" y1="-27.94" x2="-9.4615" y2="-27.94" width="0.254" layer="1"/>
 <wire x1="8.41375" y1="-7.77875" x2="6.0325" y2="-5.3975" width="1.651" layer="16"/>
@@
 <via x="2.54" y="-26.035" extent="1-16" drill="0.35"/>
 <wire x1="-3.175" y1="-26.035" x2="2.54" y2="-26.035" width="0.254" layer="16"/>
+<contactref element="R2" pad="1"/>
+<wire x1="-35" y1="-29.5" x2="-35" y2="-32.5082875" width="0.254" layer="1"/>
+<wire x1="-33.9452" y1="-34.8888" x2="-32.639" y2="-36.195" width="0.254" layer="1"/>
+<wire x1="-35" y1="-32.5082875" x2="-33.9452" y2="-33.5630875" width="0.254" layer="1"/>
+<wire x1="-33.9452" y1="-33.5630875" x2="-33.9452" y2="-34.8888" width="0.254" layer="1"/>
 </signal>
 <signal name="BT_TX">
@@
 <wire x1="-10.795" y1="-33.02" x2="-11.43" y2="-33.655" width="0.3048" layer="16"/>
 <via x="-11.43" y="-33.655" extent="1-16" drill="0.35"/>
-<wire x1="-11.43" y1="-33.655" x2="-11.43" y2="-34.29" width="0.254" layer="1"/>
-<wire x1="-11.43" y1="-34.29" x2="-13.65" y2="-36.51" width="0.254" layer="1"/>
-<wire x1="-14.14" y1="-36.51" x2="-13.65" y2="-36.51" width="0.254" layer="1"/>
+<wire x1="-12.87" y1="-31.43" x2="-12.87" y2="-32.215" width="0.254" layer="1"/>
+<wire x1="-11.43" y1="-33.655" x2="-12.87" y2="-32.215" width="0.254" layer="1"/>
 </signal>
 <signal name="SD_CD">
@@
 <contactref element="Q3" pad="2"/>
 <wire x1="-9.52425" y1="-28.3972" x2="-2.9972" y2="-28.3972" width="0.254" layer="1"/>
-<wire x1="-9.7028" y1="-28.57575" x2="-9.52425" y2="-28.3972" width="0.254" layer="1"/>
-<wire x1="-14.14" y1="-34.61" x2="-9.7028" y2="-30.1728" width="0.254" layer="1"/>
-<wire x1="-9.7028" y1="-30.1728" x2="-9.7028" y2="-28.57575" width="0.254" layer="1"/>
+<wire x1="-9.52425" y1="-28.3972" x2="-10.65705" y2="-29.53" width="0.254" layer="1"/>
+<wire x1="-12.87" y1="-29.53" x2="-10.65705" y2="-29.53" width="0.254" layer="1"/>
 <wire x1="-2.9972" y1="-28.3972" x2="0.3" y2="-25.1" width="0.254" layer="1"/>
 <wire x1="0.3" y1="-25.1" x2="0.3" y2="-23.645" width="0.254" layer="1"/>
+<contactref element="D1" pad="1"/>
+<wire x1="-13.818" y1="-35.56" x2="-12.5452" y2="-34.2872" width="0.254" layer="1"/>
+<wire x1="-12.5452" y1="-34.2872" x2="-11.16813125" y2="-34.2872" width="0.254" layer="1"/>
+<wire x1="-11.16813125" y1="-34.2872" x2="-10.65705" y2="-33.77611875" width="0.254" layer="1"/>
+<wire x1="-10.65705" y1="-33.77611875" x2="-10.65705" y2="-29.53" width="0.254" layer="1"/>
+</signal>
+<signal name="N$1">
+<contactref element="D1" pad="2"/>
+<contactref element="R2" pad="2"/>
+<wire x1="-30.861" y1="-36.195" x2="-17.297" y2="-36.195" width="0.254" layer="1"/>
+<wire x1="-17.297" y1="-36.195" x2="-16.662" y2="-35.56" width="0.254" layer="1"/>
 </signal>
 </signals>
