File: BeaconBoard2/PCBFORNICOLESAVE.sch (EAGLE design)
At the start: 108 parts, among them Q1 FDC645N, U1 ATMega2560, U2 3X3BGA0.4MM

Commit message: removed GPS PPS again lol
Parts:
- removed GPS_PPS, GPS_RX: JUMPER30V, Connectors:JUMPER30V
Connections:
- removed net GPS_FLEX: GPS_PPS.1, GPS_RX.2, R31.2, U1.P$46
- removed net GPS_PPS: GPS.1PPS, GPS_PPS.2
- net GPS_RX: now also R31.2, U1.P$46; no longer GPS_RX.1
Changed lines of the file:
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@@
 <part name="R12" library="Resistors" deviceset="RES" device="0603" value="1k"/>
 <part name="D8" library="Diodes" deviceset="DIODE" device="SOD323" value="BAT54"/>
-<part name="GPS_RX" library="Connectors" deviceset="JUMPER" device="30V"/>
-<part name="GPS_PPS" library="Connectors" deviceset="JUMPER" device="30V"/>
 <part name="C24" library="Capacitors" deviceset="CAP_NP" device="0603" value="100n"/>
 <part name="C25" library="Capacitors" deviceset="CAP_NP" device="1206" value="10u"/>
@@
 </segment>
 </net>
-<net name="GPS_FLEX" class="0">
+<net name="GPS_RX" class="0">
 <segment>
 <wire x1="71.12" y1="15.24" x2="71.12" y2="-2.54" width="0.1524" layer="91"/>
@@
 <attribute name="VALUE" x="33.02" y="60.96" size="1.016" layer="96" rot="R270" align="center"/>
 </instance>
-<instance part="GPS_RX" gate="G$1" x="43.18" y="25.4" smashed="yes">
-<attribute name="NAME" x="43.18" y="26.67" size="1.016" layer="95" align="bottom-center"/>
-</instance>
-<instance part="GPS_PPS" gate="G$1" x="83.82" y="25.4" smashed="yes">
-<attribute name="NAME" x="83.82" y="26.67" size="1.016" layer="95" align="bottom-center"/>
-</instance>
 <instance part="D20" gate="G$1" x="15.24" y="43.18" smashed="yes" rot="R90">
 <attribute name="NAME" x="13.97" y="45.72" size="1.778" layer="95" rot="R180" align="center"/>
@@
 <label x="43.18" y="40.64" size="1.778" layer="95" rot="MR0"/>
 <pinref part="GPS" gate="G$1" pin="RX"/>
-<wire x1="30.48" y1="40.64" x2="30.48" y2="25.4" width="0.1524" layer="91"/>
-<wire x1="30.48" y1="25.4" x2="40.64" y2="25.4" width="0.1524" layer="91"/>
-<pinref part="GPS_RX" gate="G$1" pin="1"/>
+<wire x1="30.48" y1="40.64" x2="30.48" y2="20.32" width="0.1524" layer="91"/>
+<wire x1="27.94" y1="20.32" x2="30.48" y2="20.32" width="0.1524" layer="91"/>
+<pinref part="R31" gate="G$1" pin="2"/>
 </segment>
 </net>
@@
 </segment>
 </net>
-<net name="GPS_PPS" class="0">
-<segment>
-<wire x1="78.74" y1="45.72" x2="96.52" y2="45.72" width="0.1524" layer="91"/>
-<label x="83.82" y="45.72" size="1.778" layer="95"/>
-<pinref part="GPS" gate="G$1" pin="1PPS"/>
-<wire x1="86.36" y1="25.4" x2="96.52" y2="25.4" width="0.1524" layer="91"/>
-<wire x1="96.52" y1="25.4" x2="96.52" y2="45.72" width="0.1524" layer="91"/>
-<pinref part="GPS_PPS" gate="G$1" pin="2"/>
-</segment>
-</net>
-<net name="GPS_FLEX" class="0">
-<segment>
-<wire x1="45.72" y1="25.4" x2="48.26" y2="25.4" width="0.1524" layer="91"/>
-<label x="58.42" y="25.4" size="1.778" layer="95"/>
-<pinref part="GPS_RX" gate="G$1" pin="2"/>
-<pinref part="GPS_PPS" gate="G$1" pin="1"/>
-<wire x1="48.26" y1="25.4" x2="81.28" y2="25.4" width="0.1524" layer="91"/>
-<wire x1="27.94" y1="20.32" x2="48.26" y2="20.32" width="0.1524" layer="91"/>
-<wire x1="48.26" y1="20.32" x2="48.26" y2="25.4" width="0.1524" layer="91"/>
-<junction x="48.26" y="25.4"/>
-<pinref part="R31" gate="G$1" pin="2"/>
-</segment>
-</net>

Commit message: removed GPS pps (again)
Parts:
- added R3: 1k, Resistors:RES0603
Connections:
- removed net SD_3V3: D1.A, Q1.S, SD.VCC
- new net SD_GND: D1.C, Q1.D, SD.GND
- net 3V3: now also R3.1, SD.VCC; no longer Q1.D
- net GND: now also Q1.S; no longer SD.GND
- net N$1: now also D1.A, R3.2; no longer D1.C, R2.1
- net SD_PWR: now also R2.1
Other:
- moved on the sheet: D1, Q1, R2
Changed lines of the file:
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@@
 <part name="Q1" library="Transistors" deviceset="NFET" device="WDFN-6" value="FDC645N"/>
 <part name="R2" library="Resistors" deviceset="RES" device="0603" value="10k"/>
+<part name="R3" library="Resistors" deviceset="RES" device="0603" value="1k"/>
 <part name="D1" library="Diodes" deviceset="LED" device="1206"/>
 <part name="D2" library="Diodes" deviceset="LED" device="1206"/>
@@
 <attribute name="NAME" x="58.42" y="43.18" size="1.4224" layer="95" align="center"/>
 </instance>
-<instance part="Q1" gate="G$1" x="-15.24" y="40.64" smashed="yes">
-<attribute name="NAME" x="-13.97" y="41.91" size="1.016" layer="95" align="center-left"/>
-<attribute name="VALUE" x="-13.97" y="39.37" size="1.016" layer="96" align="center-left"/>
-</instance>
-<instance part="R2" gate="G$1" x="-15.24" y="15.24" smashed="yes">
-<attribute name="NAME" x="-17.145" y="15.24" size="1.016" layer="95" rot="R90" align="center"/>
-<attribute name="VALUE" x="-13.335" y="15.24" size="1.016" layer="96" rot="R90" align="center"/>
-</instance>
-<instance part="D1" gate="G$1" x="-15.24" y="25.4" smashed="yes">
-<attribute name="NAME" x="-12.7" y="26.67" size="1.778" layer="95" rot="R90" align="center"/>
-<attribute name="VALUE" x="-10.16" y="26.67" size="1.778" layer="96" rot="R90" align="center"/>
+<instance part="Q1" gate="G$1" x="27.94" y="17.78" smashed="yes">
+<attribute name="NAME" x="29.21" y="19.05" size="1.016" layer="95" align="center-left"/>
+<attribute name="VALUE" x="29.21" y="16.51" size="1.016" layer="96" align="center-left"/>
+</instance>
+<instance part="R2" gate="G$1" x="17.78" y="10.16" smashed="yes">
+<attribute name="NAME" x="15.875" y="10.16" size="1.016" layer="95" rot="R90" align="center"/>
+<attribute name="VALUE" x="19.685" y="10.16" size="1.016" layer="96" rot="R90" align="center"/>
+</instance>
+<instance part="R3" gate="G$1" x="15.24" y="30.48" smashed="yes" rot="R90">
+<attribute name="NAME" x="15.24" y="28.575" size="1.016" layer="95" rot="R180" align="center"/>
+<attribute name="VALUE" x="15.24" y="32.385" size="1.016" layer="96" rot="R180" align="center"/>
+</instance>
+<instance part="D1" gate="G$1" x="22.86" y="30.48" smashed="yes" rot="R90">
+<attribute name="NAME" x="21.59" y="33.02" size="1.778" layer="95" rot="R180" align="center"/>
+<attribute name="VALUE" x="21.59" y="35.56" size="1.778" layer="96" rot="R180" align="center"/>
 </instance>
 <instance part="D2" gate="G$1" x="22.86" y="40.64" smashed="yes" rot="R90">
@@
 <net name="3V3" class="0">
 <segment>
+<pinref part="SD" gate="G$1" pin="VCC"/>
+<wire x1="43.18" y1="33.02" x2="27.94" y2="33.02" width="0.1524" layer="91"/>
+<label x="43.18" y="33.02" size="1.778" layer="95" rot="MR0"/>
+</segment>
+<segment>
 <pinref part="R4" gate="G$1" pin="1"/>
 <wire x1="12.7" y1="40.64" x2="2.54" y2="40.64" width="0.1524" layer="91"/>
@@
 </segment>
 <segment>
-<wire x1="-15.24" y1="45.72" x2="-25.4" y2="45.72" width="0.1524" layer="91"/>
-<label x="-22.86" y="45.72" size="1.778" layer="95"/>
-<pinref part="Q1" gate="G$1" pin="D"/>
+<pinref part="R3" gate="G$1" pin="1"/>
+<wire x1="12.7" y1="30.48" x2="2.54" y2="30.48" width="0.1524" layer="91"/>
+<label x="5.08" y="30.48" size="1.778" layer="95"/>
 </segment>
 </net>
@@
 <segment>
 <pinref part="SD" gate="G$1" pin="CD"/>
-<wire x1="43.18" y1="25.4" x2="27.94" y2="25.4" width="0.1524" layer="91"/>
+<wire x1="43.18" y1="25.4" x2="33.02" y2="25.4" width="0.1524" layer="91"/>
 <label x="43.18" y="25.4" size="1.778" layer="95" rot="MR0"/>
 </segment>
@@
 <segment>
 <pinref part="Q1" gate="G$1" pin="G"/>
-<wire x1="-22.86" y1="38.1" x2="-40.64" y2="38.1" width="0.1524" layer="91"/>
-<label x="-38.1" y="38.1" size="1.778" layer="95"/>
+<wire x1="20.32" y1="15.24" x2="17.78" y2="15.24" width="0.1524" layer="91"/>
+<wire x1="17.78" y1="12.7" x2="17.78" y2="15.24" width="0.1524" layer="91"/>
+<wire x1="17.78" y1="15.24" x2="2.54" y2="15.24" width="0.1524" layer="91"/>
+<pinref part="R2" gate="G$1" pin="1"/>
+<junction x="17.78" y="15.24"/>
+<label x="5.08" y="15.24" size="1.778" layer="95"/>
 </segment>
 </net>
 <net name="GND" class="0">
 <segment>
-<wire x1="-15.24" y1="2.54" x2="-15.24" y2="12.7" width="0.1524" layer="91"/>
+<pinref part="Q1" gate="G$1" pin="S"/>
+<wire x1="27.94" y1="12.7" x2="27.94" y2="5.08" width="0.1524" layer="91"/>
+<wire x1="27.94" y1="5.08" x2="17.78" y2="5.08" width="0.1524" layer="91"/>
+<wire x1="17.78" y1="5.08" x2="17.78" y2="7.62" width="0.1524" layer="91"/>
 <pinref part="R2" gate="G$1" pin="2"/>
-<label x="-15.24" y="2.54" size="1.778" layer="95"/>
-</segment>
-<segment>
-<pinref part="SD" gate="G$1" pin="GND"/>
-<wire x1="43.18" y1="30.48" x2="27.94" y2="30.48" width="0.1524" layer="91"/>
-<label x="38.1" y="30.48" size="1.778" layer="95"/>
+<label x="20.32" y="5.08" size="1.778" layer="95"/>
+</segment>
+</net>
+<net name="N$1" class="0">
+<segment>
+<pinref part="D1" gate="G$1" pin="A"/>
+<pinref part="R3" gate="G$1" pin="2"/>
+<wire x1="17.78" y1="30.48" x2="20.32" y2="30.48" width="0.1524" layer="91"/>
 </segment>
 </net>
@@
 <pinref part="D2" gate="G$1" pin="A"/>
 <wire x1="17.78" y1="40.64" x2="20.32" y2="40.64" width="0.1524" layer="91"/>
+</segment>
+</net>
+<net name="SD_GND" class="0">
+<segment>
+<pinref part="Q1" gate="G$1" pin="D"/>
+<wire x1="27.94" y1="22.86" x2="27.94" y2="30.48" width="0.1524" layer="91"/>
+<pinref part="D1" gate="G$1" pin="C"/>
+<wire x1="25.4" y1="30.48" x2="27.94" y2="30.48" width="0.1524" layer="91"/>
+<pinref part="SD" gate="G$1" pin="GND"/>
+<wire x1="27.94" y1="30.48" x2="43.18" y2="30.48" width="0.1524" layer="91"/>
+<junction x="27.94" y="30.48"/>
+<label x="43.18" y="30.48" size="1.778" layer="95" rot="MR0"/>
 </segment>
 </net>
@@
 </segment>
 </net>
-<net name="N$1" class="0">
-<segment>
-<pinref part="D1" gate="G$1" pin="C"/>
-<pinref part="R2" gate="G$1" pin="1"/>
-<wire x1="-15.24" y1="22.86" x2="-15.24" y2="17.78" width="0.1524" layer="91"/>
-</segment>
-</net>
-<net name="SD_3V3" class="0">
-<segment>
-<pinref part="SD" gate="G$1" pin="VCC"/>
-<label x="35.56" y="33.02" size="1.778" layer="95"/>
-<pinref part="Q1" gate="G$1" pin="S"/>
-<pinref part="D1" gate="G$1" pin="A"/>
-<wire x1="-15.24" y1="35.56" x2="-15.24" y2="33.02" width="0.1524" layer="91"/>
-<wire x1="-15.24" y1="33.02" x2="-15.24" y2="27.94" width="0.1524" layer="91"/>
-<wire x1="43.18" y1="33.02" x2="-15.24" y2="33.02" width="0.1524" layer="91"/>
-<junction x="-15.24" y="33.02"/>
-</segment>
-</net>

Commit message: finished routing, fixed DRC errors and wire stubs, moved components to make soldering easier
Parts:
- removed D1: (no value), Diodes:LED1206
- removed Q1: FDC645N, Transistors:NFETWDFN-6
- removed R3: 1k, Resistors:RES0603
- added Q3: FDN340P, FDN340P:FDN340P
Connections:
- removed net SD_GND: D1.C, Q1.D, SD.GND
- new net SD_3V3: SD.VCC
- net 3V3: now also Q3.D; no longer R3.1, SD.VCC
- net GND: now also SD.GND; no longer Q1.S
- net N$1: now also Q3.S, R2.1; no longer D1.A, R3.2
- net SD_PWR: now also Q3.G; no longer Q1.G, R2.1
Other:
- moved on the sheet: R2
Changed lines of the file:
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@@
 <part name="Y1" library="Chips" deviceset="XRES" device="1206"/>
 <part name="SD" library="Connectors" deviceset="MICROSD" device="FRONT"/>
-<part name="Q1" library="Transistors" deviceset="NFET" device="WDFN-6" value="FDC645N"/>
 <part name="R2" library="Resistors" deviceset="RES" device="0603" value="10k"/>
-<part name="R3" library="Resistors" deviceset="RES" device="0603" value="1k"/>
-<part name="D1" library="Diodes" deviceset="LED" device="1206"/>
 <part name="D2" library="Diodes" deviceset="LED" device="1206"/>
 <part name="R4" library="Resistors" deviceset="RES" device="0603" value="1k"/>
@@
 <part name="R25" library="Resistors" deviceset="RES" device="0603" value="1k"/>
 <part name="SOL1" library="Connectors" deviceset="PINHD-1X2" device="/90"/>
+<part name="Q3" library="FDN340P" deviceset="FDN340P" device=""/>
 </parts>
 <sheets>
@@
 <attribute name="NAME" x="58.42" y="43.18" size="1.4224" layer="95" align="center"/>
 </instance>
-<instance part="Q1" gate="G$1" x="27.94" y="17.78" smashed="yes">
-<attribute name="NAME" x="29.21" y="19.05" size="1.016" layer="95" align="center-left"/>
-<attribute name="VALUE" x="29.21" y="16.51" size="1.016" layer="96" align="center-left"/>
-</instance>
-<instance part="R2" gate="G$1" x="17.78" y="10.16" smashed="yes">
-<attribute name="NAME" x="15.875" y="10.16" size="1.016" layer="95" rot="R90" align="center"/>
-<attribute name="VALUE" x="19.685" y="10.16" size="1.016" layer="96" rot="R90" align="center"/>
-</instance>
-<instance part="R3" gate="G$1" x="15.24" y="30.48" smashed="yes" rot="R90">
-<attribute name="NAME" x="15.24" y="28.575" size="1.016" layer="95" rot="R180" align="center"/>
-<attribute name="VALUE" x="15.24" y="32.385" size="1.016" layer="96" rot="R180" align="center"/>
-</instance>
-<instance part="D1" gate="G$1" x="22.86" y="30.48" smashed="yes" rot="R90">
-<attribute name="NAME" x="21.59" y="33.02" size="1.778" layer="95" rot="R180" align="center"/>
-<attribute name="VALUE" x="21.59" y="35.56" size="1.778" layer="96" rot="R180" align="center"/>
+<instance part="R2" gate="G$1" x="12.7" y="15.24" smashed="yes">
+<attribute name="NAME" x="10.795" y="15.24" size="1.016" layer="95" rot="R90" align="center"/>
+<attribute name="VALUE" x="14.605" y="15.24" size="1.016" layer="96" rot="R90" align="center"/>
 </instance>
 <instance part="D2" gate="G$1" x="22.86" y="40.64" smashed="yes" rot="R90">
@@
 <attribute name="NAME" x="15.24" y="38.735" size="1.016" layer="95" rot="R180" align="center"/>
 <attribute name="VALUE" x="15.24" y="42.545" size="1.016" layer="96" rot="R180" align="center"/>
+</instance>
+<instance part="Q3" gate="G$1" x="12.7" y="25.4" smashed="yes">
+<attribute name="VALUE" x="15.24135" y="22.85865" size="1.778940625" layer="96"/>
+<attribute name="NAME" x="15.2401" y="25.4" size="1.77806875" layer="95"/>
 </instance>
 </instances>
@@
 <net name="3V3" class="0">
 <segment>
-<pinref part="SD" gate="G$1" pin="VCC"/>
-<wire x1="43.18" y1="33.02" x2="27.94" y2="33.02" width="0.1524" layer="91"/>
-<label x="43.18" y="33.02" size="1.778" layer="95" rot="MR0"/>
-</segment>
-<segment>
 <pinref part="R4" gate="G$1" pin="1"/>
 <wire x1="12.7" y1="40.64" x2="2.54" y2="40.64" width="0.1524" layer="91"/>
@@
 </segment>
 <segment>
-<pinref part="R3" gate="G$1" pin="1"/>
 <wire x1="12.7" y1="30.48" x2="2.54" y2="30.48" width="0.1524" layer="91"/>
 <label x="5.08" y="30.48" size="1.778" layer="95"/>
+<pinref part="Q3" gate="G$1" pin="D"/>
 </segment>
 </net>
@@
 <net name="SD_PWR" class="0">
 <segment>
-<pinref part="Q1" gate="G$1" pin="G"/>
-<wire x1="20.32" y1="15.24" x2="17.78" y2="15.24" width="0.1524" layer="91"/>
-<wire x1="17.78" y1="12.7" x2="17.78" y2="15.24" width="0.1524" layer="91"/>
-<wire x1="17.78" y1="15.24" x2="2.54" y2="15.24" width="0.1524" layer="91"/>
-<pinref part="R2" gate="G$1" pin="1"/>
-<junction x="17.78" y="15.24"/>
-<label x="5.08" y="15.24" size="1.778" layer="95"/>
+<pinref part="Q3" gate="G$1" pin="G"/>
+<wire x1="7.62" y1="22.86" x2="2.54" y2="22.86" width="0.1524" layer="91"/>
+<label x="-2.54" y="22.86" size="1.778" layer="95"/>
 </segment>
 </net>
 <net name="GND" class="0">
 <segment>
-<pinref part="Q1" gate="G$1" pin="S"/>
-<wire x1="27.94" y1="12.7" x2="27.94" y2="5.08" width="0.1524" layer="91"/>
-<wire x1="27.94" y1="5.08" x2="17.78" y2="5.08" width="0.1524" layer="91"/>
-<wire x1="17.78" y1="5.08" x2="17.78" y2="7.62" width="0.1524" layer="91"/>
+<pinref part="SD" gate="G$1" pin="GND"/>
+<wire x1="43.18" y1="30.48" x2="27.94" y2="30.48" width="0.1524" layer="91"/>
+<label x="38.1" y="30.48" size="1.778" layer="95"/>
+</segment>
+<segment>
 <pinref part="R2" gate="G$1" pin="2"/>
-<label x="20.32" y="5.08" size="1.778" layer="95"/>
-</segment>
-</net>
-<net name="N$1" class="0">
-<segment>
-<pinref part="D1" gate="G$1" pin="A"/>
-<pinref part="R3" gate="G$1" pin="2"/>
-<wire x1="17.78" y1="30.48" x2="20.32" y2="30.48" width="0.1524" layer="91"/>
+<wire x1="12.7" y1="12.7" x2="12.7" y2="5.08" width="0.1524" layer="91"/>
+<label x="7.62" y="10.16" size="1.778" layer="95"/>
 </segment>
 </net>
@@
 <pinref part="D2" gate="G$1" pin="A"/>
 <wire x1="17.78" y1="40.64" x2="20.32" y2="40.64" width="0.1524" layer="91"/>
-</segment>
-</net>
-<net name="SD_GND" class="0">
-<segment>
-<pinref part="Q1" gate="G$1" pin="D"/>
-<wire x1="27.94" y1="22.86" x2="27.94" y2="30.48" width="0.1524" layer="91"/>
-<pinref part="D1" gate="G$1" pin="C"/>
-<wire x1="25.4" y1="30.48" x2="27.94" y2="30.48" width="0.1524" layer="91"/>
-<pinref part="SD" gate="G$1" pin="GND"/>
-<wire x1="27.94" y1="30.48" x2="43.18" y2="30.48" width="0.1524" layer="91"/>
-<junction x="27.94" y="30.48"/>
-<label x="43.18" y="30.48" size="1.778" layer="95" rot="MR0"/>
 </segment>
 </net>
@@
 </segment>
 </net>
+<net name="SD_3V3" class="0">
+<segment>
+<pinref part="SD" gate="G$1" pin="VCC"/>
+<wire x1="43.18" y1="33.02" x2="27.94" y2="33.02" width="0.1524" layer="91"/>
+<label x="33.02" y="33.02" size="1.778" layer="95"/>
+</segment>
+</net>
+<net name="N$1" class="0">
+<segment>
+<pinref part="Q3" gate="G$1" pin="S"/>
+<pinref part="R2" gate="G$1" pin="1"/>
+<wire x1="12.7" y1="20.32" x2="12.7" y2="17.78" width="0.1524" layer="91"/>
+</segment>
+</net>

Commit message: rerouted sd card slightly to fix mistake
Parts:
- removed R2: 10k, Resistors:RES0603
Connections:
- removed net N$1: Q3.S, R2.1
- net GND: no longer R2.2
- net SD_3V3: now also Q3.S
Changed lines of the file:
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@@
 <part name="Y1" library="Chips" deviceset="XRES" device="1206"/>
 <part name="SD" library="Connectors" deviceset="MICROSD" device="FRONT"/>
-<part name="R2" library="Resistors" deviceset="RES" device="0603" value="10k"/>
 <part name="D2" library="Diodes" deviceset="LED" device="1206"/>
 <part name="R4" library="Resistors" deviceset="RES" device="0603" value="1k"/>
@@
 <attribute name="NAME" x="58.42" y="43.18" size="1.4224" layer="95" align="center"/>
 </instance>
-<instance part="R2" gate="G$1" x="12.7" y="15.24" smashed="yes">
-<attribute name="NAME" x="10.795" y="15.24" size="1.016" layer="95" rot="R90" align="center"/>
-<attribute name="VALUE" x="14.605" y="15.24" size="1.016" layer="96" rot="R90" align="center"/>
-</instance>
 <instance part="D2" gate="G$1" x="22.86" y="40.64" smashed="yes" rot="R90">
 <attribute name="NAME" x="21.59" y="43.18" size="1.778" layer="95" rot="R180" align="center"/>
@@
 <label x="38.1" y="30.48" size="1.778" layer="95"/>
 </segment>
-<segment>
-<pinref part="R2" gate="G$1" pin="2"/>
-<wire x1="12.7" y1="12.7" x2="12.7" y2="5.08" width="0.1524" layer="91"/>
-<label x="7.62" y="10.16" size="1.778" layer="95"/>
-</segment>
 </net>
 <net name="N$4" class="0">
@@
 <segment>
 <pinref part="SD" gate="G$1" pin="VCC"/>
-<wire x1="43.18" y1="33.02" x2="27.94" y2="33.02" width="0.1524" layer="91"/>
+<wire x1="43.18" y1="33.02" x2="25.4" y2="33.02" width="0.1524" layer="91"/>
 <label x="33.02" y="33.02" size="1.778" layer="95"/>
-</segment>
-</net>
-<net name="N$1" class="0">
-<segment>
 <pinref part="Q3" gate="G$1" pin="S"/>
-<pinref part="R2" gate="G$1" pin="1"/>
 <wire x1="12.7" y1="20.32" x2="12.7" y2="17.78" width="0.1524" layer="91"/>
-</segment>
-</net>
+<wire x1="12.7" y1="17.78" x2="25.4" y2="17.78" width="0.1524" layer="91"/>
+<wire x1="25.4" y1="17.78" x2="25.4" y2="33.02" width="0.1524" layer="91"/>
+</segment>
+</net>

Commit message: fixed sd card mosfet
Parts:
- added D1: (no value), Diodes:LED1206
- added R2: 1k, Resistors:RES0603
Connections:
- new net N$1: D1.C, R2.2
- net GND: now also R2.1
- net SD_3V3: now also D1.A
Changed lines of the file:
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@@
 <part name="SOL1" library="Connectors" deviceset="PINHD-1X2" device="/90"/>
 <part name="Q3" library="FDN340P" deviceset="FDN340P" device=""/>
+<part name="D1" library="Diodes" deviceset="LED" device="1206"/>
+<part name="R2" library="Resistors" deviceset="RES" device="0603" value="1k"/>
 </parts>
 <sheets>
@@
 <attribute name="NAME" x="15.2401" y="25.4" size="1.77806875" layer="95"/>
 </instance>
+<instance part="D1" gate="G$1" x="12.7" y="15.24" smashed="yes">
+<attribute name="NAME" x="15.24" y="16.51" size="1.778" layer="95" rot="R90" align="center"/>
+<attribute name="VALUE" x="17.78" y="16.51" size="1.778" layer="96" rot="R90" align="center"/>
+</instance>
+<instance part="R2" gate="G$1" x="12.7" y="7.62" smashed="yes" rot="R180">
+<attribute name="NAME" x="14.605" y="7.62" size="1.016" layer="95" rot="R270" align="center"/>
+<attribute name="VALUE" x="10.795" y="7.62" size="1.016" layer="96" rot="R270" align="center"/>
+</instance>
 </instances>
 <busses>
@@
 <wire x1="43.18" y1="30.48" x2="27.94" y2="30.48" width="0.1524" layer="91"/>
 <label x="38.1" y="30.48" size="1.778" layer="95"/>
+</segment>
+<segment>
+<pinref part="R2" gate="G$1" pin="1"/>
+<wire x1="12.7" y1="5.08" x2="12.7" y2="0" width="0.1524" layer="91"/>
+<label x="7.62" y="0" size="1.778" layer="95"/>
 </segment>
 </net>
@@
 <wire x1="12.7" y1="17.78" x2="25.4" y2="17.78" width="0.1524" layer="91"/>
 <wire x1="25.4" y1="17.78" x2="25.4" y2="33.02" width="0.1524" layer="91"/>
-</segment>
-</net>
+<pinref part="D1" gate="G$1" pin="A"/>
+<junction x="12.7" y="17.78"/>
+</segment>
+</net>
+<net name="N$1" class="0">
+<segment>
+<pinref part="D1" gate="G$1" pin="C"/>
+<pinref part="R2" gate="G$1" pin="2"/>
+<wire x1="12.7" y1="12.7" x2="12.7" y2="10.16" width="0.1524" layer="91"/>
+</segment>
+</net>
